File: keyboard/_autosave-keyboard.kicad_pcb (KiCad board)
At the start: 2 copper layers, 356 parts, among them K1 KEYSW, K10 KEYSW, K100 KEYSW, K101 KEYSW, K102 KEYSW, K103 KEYSW, K104 KEYSW, K11 KEYSW, K12 KEYSW, K13 KEYSW, K14 KEYSW, K15 KEYSW, K16 KEYSW, K17 KEYSW, K18 KEYSW, K19 KEYSW, K2 KEYSW, K20 KEYSW, K21 KEYSW, K22 KEYSW, K23 KEYSW, K24 KEYSW, K25 KEYSW, K26 KEYSW, K27 KEYSW, K28 KEYSW, K29 KEYSW, K3 KEYSW, K30 KEYSW, K31 KEYSW, K32 KEYSW, K33 KEYSW, K34 KEYSW, K35 KEYSW, K36 KEYSW, K37 KEYSW, K38 KEYSW, K39 KEYSW, K4 KEYSW, K40 KEYSW, K41 KEYSW, K42 KEYSW, K43 KEYSW, K44 KEYSW, K45 KEYSW, K46 KEYSW, K47 KEYSW, K48 KEYSW, K49 KEYSW, K5 KEYSW, K50 KEYSW, K51 KEYSW, K52 KEYSW, K53 KEYSW, K54 KEYSW, K55 KEYSW, K56 KEYSW, K57 KEYSW, K58 KEYSW, K59 KEYSW, K6 KEYSW, K60 KEYSW, K61 KEYSW, K62 KEYSW, K63 KEYSW, K64 KEYSW, K65 KEYSW, K66 KEYSW, K67 KEYSW, K68 KEYSW, K69 KEYSW, K7 KEYSW, K70 KEYSW, K71 KEYSW, K72 KEYSW, K73 KEYSW, K74 KEYSW, K75 KEYSW, K76 KEYSW, K77 KEYSW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

Commit message: add switches/leds
Parts:
- D105, D106, D107, D108, D109, D110, D111, D112, D113, D114, D115, D116, D117, D118, D119, D120, D121, D122, D123, D124, D125, D126, D127, D128, D129, D130, D131, D132, D133, D134, D135, D136, D137, D138, D139, D140, D141, D142, D143, D144, D145, D146, D147, D148, D149, D150, D151, D152, D153, D154, D155, D156, D157, D158, D159, D160, D161, D162, D163, D164, D165, D166, D167, D168, D169, D170, D171, D172, D173, D174, D175, D176, D177, D178, D179, D180, D181, D182, D183, D184, D185, D186, D187, D188, D189, D190, D191, D192, D193, D194, D195, D196, D197, D198, D199, D200, D201, D202, D203, D204, D205, D206, D207, D208, D209, D210, D211, D212, D213, D214, D215, D216, D217, D218, D219, D220, D221, D222, D223, D224, D225, D226, D227, D228, D229, D230, D231, D232: value WS2812B -> SK6812MINI; footprint LED_SMD:LED_WS2812B_PLCC4_5.0x5.0mm_P3.2mm -> LED_SMD:LED_SK6812MINI_PLCC4_3.5x3.5mm_P1.75mm
- moved R2 361.5 mm to (386.2, 74.0)
- moved R3 358.2 mm to (388.3, 76.9)
- moved R4 353.1 mm to (388.3, 79.9)
- moved R5 347.9 mm to (388.3, 82.8)
- moved SW2 347.1 mm to (344.9, 73.8)
- moved R6 342.7 mm to (388.3, 85.8)
- moved R7 337.5 mm to (388.3, 88.7)
- moved C1 327.0 mm to (387.2, 92.1)
- moved D38 318.9 mm to (366.0, 52.1)
- moved C8 318.6 mm to (344.0, 107.0)
- moved C5 317.8 mm to (387.2, 95.1)
- moved D81 315.8 mm to (376.4, 52.1)
- moved D79 297.2 mm to (366.0, 59.3)
- moved D80 295.8 mm to (366.0, 55.7)
- moved C7 294.6 mm to (328.1, 122.3)
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Connections:
- D105 pad 1: VCC -> Net-(D105-Pad1)
- D105 pad 2: Net-(D105-Pad2) -> GND
- D105 pad 3: GND -> /LEDDATA
- D105 pad 4: /LEDDATA -> VCC
- D106 pad 1: VCC -> Net-(D106-Pad1)
- D106 pad 2: Net-(D106-Pad2) -> GND
- D106 pad 3: GND -> Net-(D106-Pad3)
- D106 pad 4: Net-(D106-Pad4) -> VCC
- D107 pad 1: VCC -> Net-(D107-Pad1)
- D107 pad 2: Net-(D107-Pad2) -> GND
- D107 pad 3: GND -> Net-(D107-Pad3)
- D107 pad 4: Net-(D107-Pad4) -> VCC
- D108 pad 1: VCC -> Net-(D108-Pad1)
- D108 pad 2: Net-(D108-Pad2) -> GND
- D108 pad 3: GND -> Net-(D108-Pad3)
- D108 pad 4: Net-(D108-Pad4) -> VCC
- D109 pad 1: VCC -> Net-(D109-Pad1)
- D109 pad 2: Net-(D109-Pad2) -> GND
- D109 pad 3: GND -> Net-(D109-Pad3)
- D109 pad 4: Net-(D109-Pad4) -> VCC
- D110 pad 1: VCC -> Net-(D110-Pad1)
- D110 pad 2: Net-(D110-Pad2) -> GND
- D110 pad 3: GND -> Net-(D110-Pad3)
- D110 pad 4: Net-(D110-Pad4) -> VCC
- D111 pad 1: VCC -> Net-(D111-Pad1)
- D111 pad 2: Net-(D111-Pad2) -> GND
- D111 pad 3: GND -> Net-(D111-Pad3)
- D111 pad 4: Net-(D111-Pad4) -> VCC
- D112 pad 1: VCC -> Net-(D112-Pad1)
- D112 pad 2: Net-(D112-Pad2) -> GND
- D112 pad 3: GND -> Net-(D112-Pad3)
- D112 pad 4: Net-(D112-Pad4) -> VCC
- D113 pad 1: VCC -> Net-(D113-Pad1)
- D113 pad 2: Net-(D113-Pad2) -> GND
- D113 pad 3: GND -> Net-(D105-Pad1)
- D113 pad 4: Net-(D105-Pad2) -> VCC
- D114 pad 1: VCC -> Net-(D114-Pad1)
- D114 pad 2: Net-(D114-Pad2) -> GND
- D114 pad 3: GND -> Net-(D106-Pad1)
- D114 pad 4: Net-(D106-Pad2) -> VCC
- D115 pad 1: VCC -> Net-(D115-Pad1)
- D115 pad 2: Net-(D115-Pad2) -> GND
- D115 pad 3: GND -> Net-(D107-Pad1)
- D115 pad 4: Net-(D107-Pad2) -> VCC
- D116 pad 1: VCC -> Net-(D116-Pad1)
- D116 pad 2: Net-(D116-Pad2) -> GND
- D116 pad 3: GND -> Net-(D108-Pad1)
- D116 pad 4: Net-(D108-Pad2) -> VCC
- D117 pad 1: VCC -> Net-(D117-Pad1)
- D117 pad 2: Net-(D117-Pad2) -> GND
- D117 pad 3: GND -> Net-(D109-Pad1)
- D117 pad 4: Net-(D109-Pad2) -> VCC
- D118 pad 1: VCC -> Net-(D118-Pad1)
- D118 pad 2: Net-(D118-Pad2) -> GND
- D118 pad 3: GND -> Net-(D110-Pad1)
- D118 pad 4: Net-(D110-Pad2) -> VCC
- D119 pad 1: VCC -> Net-(D119-Pad1)
- D119 pad 2: Net-(D119-Pad2) -> GND
- D119 pad 3: GND -> Net-(D111-Pad1)
- D119 pad 4: Net-(D111-Pad2) -> VCC
- D120 pad 1: VCC -> Net-(D120-Pad1)
- D120 pad 2: Net-(D120-Pad2) -> GND
- D120 pad 3: GND -> Net-(D112-Pad1)
- D120 pad 4: Net-(D112-Pad2) -> VCC
- D121 pad 1: VCC -> Net-(D121-Pad1)
- D121 pad 2: Net-(D121-Pad2) -> GND
- D121 pad 3: GND -> Net-(D113-Pad1)
- D121 pad 4: Net-(D113-Pad2) -> VCC
- D122 pad 1: VCC -> Net-(D122-Pad1)
- D122 pad 2: Net-(D122-Pad2) -> GND
- D122 pad 3: GND -> Net-(D114-Pad1)
- D122 pad 4: Net-(D114-Pad2) -> VCC
- D123 pad 1: VCC -> Net-(D123-Pad1)
- D123 pad 2: Net-(D123-Pad2) -> GND
- D123 pad 3: GND -> Net-(D115-Pad1)
- D123 pad 4: Net-(D115-Pad2) -> VCC
- D124 pad 1: VCC -> Net-(D124-Pad1)
- D124 pad 2: Net-(D124-Pad2) -> GND
- D124 pad 3: GND -> Net-(D116-Pad1)
- D124 pad 4: Net-(D116-Pad2) -> VCC
- D125 pad 1: VCC -> Net-(D125-Pad1)
- D125 pad 2: Net-(D125-Pad2) -> GND
- D125 pad 3: GND -> Net-(D117-Pad1)
- D125 pad 4: Net-(D117-Pad2) -> VCC
- D126 pad 1: VCC -> Net-(D126-Pad1)
- D126 pad 2: Net-(D126-Pad2) -> GND
- D126 pad 3: GND -> Net-(D118-Pad1)
- D126 pad 4: Net-(D118-Pad2) -> VCC
- D127 pad 1: VCC -> Net-(D127-Pad1)
- D127 pad 2: Net-(D127-Pad2) -> GND
- D127 pad 3: GND -> Net-(D119-Pad1)
- D127 pad 4: Net-(D119-Pad2) -> VCC
- D128 pad 1: VCC -> Net-(D128-Pad1)
- D128 pad 2: Net-(D128-Pad2) -> GND
- D128 pad 3: GND -> Net-(D120-Pad1)
- D128 pad 4: Net-(D120-Pad2) -> VCC
- D129 pad 1: VCC -> Net-(D129-Pad1)
- D129 pad 2: Net-(D129-Pad2) -> GND
- D129 pad 3: GND -> Net-(D121-Pad1)
- D129 pad 4: Net-(D121-Pad2) -> VCC
- D130 pad 1: VCC -> Net-(D130-Pad1)
- D130 pad 2: Net-(D130-Pad2) -> GND
- D130 pad 3: GND -> Net-(D122-Pad1)
- D130 pad 4: Net-(D122-Pad2) -> VCC
- D131 pad 1: VCC -> Net-(D131-Pad1)
- D131 pad 2: Net-(D131-Pad2) -> GND
- D131 pad 3: GND -> Net-(D123-Pad1)
- D131 pad 4: Net-(D123-Pad2) -> VCC
- D132 pad 1: VCC -> Net-(D132-Pad1)
- D132 pad 2: Net-(D132-Pad2) -> GND
- D132 pad 3: GND -> Net-(D124-Pad1)
- D132 pad 4: Net-(D124-Pad2) -> VCC
- D133 pad 1: VCC -> Net-(D133-Pad1)
- D133 pad 2: Net-(D133-Pad2) -> GND
- D133 pad 3: GND -> Net-(D125-Pad1)
- D133 pad 4: Net-(D125-Pad2) -> VCC
- D134 pad 1: VCC -> Net-(D134-Pad1)
- D134 pad 2: Net-(D134-Pad2) -> GND
- D134 pad 3: GND -> Net-(D126-Pad1)
- D134 pad 4: Net-(D126-Pad2) -> VCC
- D135 pad 1: VCC -> Net-(D135-Pad1)
- D135 pad 2: Net-(D135-Pad2) -> GND
- D135 pad 3: GND -> Net-(D127-Pad1)
- D135 pad 4: Net-(D127-Pad2) -> VCC
- D136 pad 1: VCC -> Net-(D136-Pad1)
- D136 pad 2: Net-(D136-Pad2) -> GND
- D136 pad 3: GND -> Net-(D128-Pad1)
- D136 pad 4: Net-(D128-Pad2) -> VCC
- D137 pad 1: VCC -> Net-(D137-Pad1)
- D137 pad 2: Net-(D137-Pad2) -> GND
- D137 pad 3: GND -> Net-(D129-Pad1)
- D137 pad 4: Net-(D129-Pad2) -> VCC
- D138 pad 1: VCC -> Net-(D138-Pad1)
- D138 pad 2: Net-(D138-Pad2) -> GND
- D138 pad 3: GND -> Net-(D130-Pad1)
- D138 pad 4: Net-(D130-Pad2) -> VCC
- D139 pad 1: VCC -> Net-(D139-Pad1)
- D139 pad 2: Net-(D139-Pad2) -> GND
- D139 pad 3: GND -> Net-(D131-Pad1)
- D139 pad 4: Net-(D131-Pad2) -> VCC
- D140 pad 1: VCC -> Net-(D140-Pad1)
- D140 pad 2: Net-(D140-Pad2) -> GND
- D140 pad 3: GND -> Net-(D132-Pad1)
- D140 pad 4: Net-(D132-Pad2) -> VCC
- D141 pad 1: VCC -> Net-(D141-Pad1)
- D141 pad 2: Net-(D141-Pad2) -> GND
- D141 pad 3: GND -> Net-(D133-Pad1)
- D141 pad 4: Net-(D133-Pad2) -> VCC
- D142 pad 1: VCC -> Net-(D142-Pad1)
- D142 pad 2: Net-(D142-Pad2) -> GND
- D142 pad 3: GND -> Net-(D134-Pad1)
- D142 pad 4: Net-(D134-Pad2) -> VCC
- D143 pad 1: VCC -> Net-(D143-Pad1)
- D143 pad 2: Net-(D143-Pad2) -> GND
- D143 pad 3: GND -> Net-(D135-Pad1)
- D143 pad 4: Net-(D135-Pad2) -> VCC
- D144 pad 1: VCC -> Net-(D144-Pad1)
- D144 pad 2: Net-(D144-Pad2) -> GND
- D144 pad 3: GND -> Net-(D136-Pad1)
- D144 pad 4: Net-(D136-Pad2) -> VCC
- D145 pad 1: VCC -> Net-(D145-Pad1)
- D145 pad 2: Net-(D145-Pad2) -> GND
- D145 pad 3: GND -> Net-(D137-Pad1)
- D145 pad 4: Net-(D137-Pad2) -> VCC
- D146 pad 1: VCC -> Net-(D146-Pad1)
- D146 pad 2: Net-(D146-Pad2) -> GND
- D146 pad 3: GND -> Net-(D138-Pad1)
- D146 pad 4: Net-(D138-Pad2) -> VCC
- D147 pad 1: VCC -> Net-(D147-Pad1)
- D147 pad 2: Net-(D147-Pad2) -> GND
- D147 pad 3: GND -> Net-(D139-Pad1)
- D147 pad 4: Net-(D139-Pad2) -> VCC
- D148 pad 1: VCC -> Net-(D148-Pad1)
- D148 pad 2: Net-(D148-Pad2) -> GND
- D148 pad 3: GND -> Net-(D140-Pad1)
- D148 pad 4: Net-(D140-Pad2) -> VCC
- D149 pad 1: VCC -> Net-(D149-Pad1)
- D149 pad 2: Net-(D149-Pad2) -> GND
- D149 pad 3: GND -> Net-(D141-Pad1)
- D149 pad 4: Net-(D141-Pad2) -> VCC
- D150 pad 1: VCC -> Net-(D150-Pad1)
- D150 pad 2: Net-(D150-Pad2) -> GND
- D150 pad 3: GND -> Net-(D142-Pad1)
- D150 pad 4: Net-(D142-Pad2) -> VCC
- D151 pad 1: VCC -> Net-(D151-Pad1)
- D151 pad 2: Net-(D151-Pad2) -> GND
- D151 pad 3: GND -> Net-(D143-Pad1)
- D151 pad 4: Net-(D143-Pad2) -> VCC
- D152 pad 1: VCC -> Net-(D152-Pad1)
- D152 pad 2: Net-(D152-Pad2) -> GND
- D152 pad 3: GND -> Net-(D144-Pad1)
- D152 pad 4: Net-(D144-Pad2) -> VCC
- D153 pad 1: VCC -> Net-(D153-Pad1)
- D153 pad 2: Net-(D153-Pad2) -> GND
- D153 pad 3: GND -> Net-(D145-Pad1)
- D153 pad 4: Net-(D145-Pad2) -> VCC
- D154 pad 1: VCC -> Net-(D154-Pad1)
- D154 pad 2: Net-(D154-Pad2) -> GND
- D154 pad 3: GND -> Net-(D146-Pad1)
- D154 pad 4: Net-(D146-Pad2) -> VCC
- D155 pad 1: VCC -> Net-(D155-Pad1)
- D155 pad 2: Net-(D155-Pad2) -> GND
- D155 pad 3: GND -> Net-(D147-Pad1)
- D155 pad 4: Net-(D147-Pad2) -> VCC
- D156 pad 1: VCC -> Net-(D156-Pad1)
- D156 pad 2: Net-(D156-Pad2) -> GND
- D156 pad 3: GND -> Net-(D148-Pad1)
- D156 pad 4: Net-(D148-Pad2) -> VCC
- D157 pad 1: VCC -> Net-(D157-Pad1)
- D157 pad 2: Net-(D157-Pad2) -> GND
- D157 pad 3: GND -> Net-(D149-Pad1)
- D157 pad 4: Net-(D149-Pad2) -> VCC
- D158 pad 1: VCC -> Net-(D158-Pad1)
- D158 pad 2: Net-(D158-Pad2) -> GND
- D158 pad 3: GND -> Net-(D150-Pad1)
- D158 pad 4: Net-(D150-Pad2) -> VCC
- D159 pad 1: VCC -> Net-(D159-Pad1)
- D159 pad 2: Net-(D159-Pad2) -> GND
- D159 pad 3: GND -> Net-(D151-Pad1)
- D159 pad 4: Net-(D151-Pad2) -> VCC
- D160 pad 1: VCC -> Net-(D160-Pad1)
- D160 pad 2: Net-(D160-Pad2) -> GND
- D160 pad 3: GND -> Net-(D152-Pad1)
- D160 pad 4: Net-(D152-Pad2) -> VCC
- D161 pad 1: VCC -> Net-(D161-Pad1)
- D161 pad 2: Net-(D161-Pad2) -> GND
- D161 pad 3: GND -> Net-(D153-Pad1)
- D161 pad 4: Net-(D153-Pad2) -> VCC
- D162 pad 1: VCC -> Net-(D162-Pad1)
- D162 pad 2: Net-(D162-Pad2) -> GND
- D162 pad 3: GND -> Net-(D154-Pad1)
- D162 pad 4: Net-(D154-Pad2) -> VCC
- D163 pad 1: VCC -> Net-(D163-Pad1)
- D163 pad 2: Net-(D163-Pad2) -> GND
- D163 pad 3: GND -> Net-(D155-Pad1)
- D163 pad 4: Net-(D155-Pad2) -> VCC
- D164 pad 1: VCC -> Net-(D164-Pad1)
- D164 pad 2: Net-(D164-Pad2) -> GND
- D164 pad 3: GND -> Net-(D156-Pad1)
- D164 pad 4: Net-(D156-Pad2) -> VCC
- D165 pad 1: VCC -> Net-(D165-Pad1)
- D165 pad 2: Net-(D165-Pad2) -> GND
- D165 pad 3: GND -> Net-(D157-Pad1)
- D165 pad 4: Net-(D157-Pad2) -> VCC
- D166 pad 1: VCC -> Net-(D166-Pad1)
- D166 pad 2: Net-(D166-Pad2) -> GND
- D166 pad 3: GND -> Net-(D158-Pad1)
- D166 pad 4: Net-(D158-Pad2) -> VCC
- D167 pad 1: VCC -> Net-(D167-Pad1)
- D167 pad 2: Net-(D167-Pad2) -> GND
- D167 pad 3: GND -> Net-(D159-Pad1)
- D167 pad 4: Net-(D159-Pad2) -> VCC
- D168 pad 1: VCC -> Net-(D168-Pad1)
- D168 pad 2: Net-(D168-Pad2) -> GND
- D168 pad 3: GND -> Net-(D160-Pad1)
- D168 pad 4: Net-(D160-Pad2) -> VCC
- D169 pad 1: VCC -> Net-(D169-Pad1)
- D169 pad 2: Net-(D169-Pad2) -> GND
- D169 pad 3: GND -> Net-(D161-Pad1)
- D169 pad 4: Net-(D161-Pad2) -> VCC
- D170 pad 1: VCC -> Net-(D170-Pad1)
- D170 pad 2: Net-(D170-Pad2) -> GND
- D170 pad 3: GND -> Net-(D162-Pad1)
- D170 pad 4: Net-(D162-Pad2) -> VCC
- D171 pad 1: VCC -> Net-(D171-Pad1)
- D171 pad 2: Net-(D171-Pad2) -> GND
- D171 pad 3: GND -> Net-(D163-Pad1)
- D171 pad 4: Net-(D163-Pad2) -> VCC
- D172 pad 1: VCC -> Net-(D172-Pad1)
- D172 pad 2: Net-(D172-Pad2) -> GND
- D172 pad 3: GND -> Net-(D164-Pad1)
- D172 pad 4: Net-(D164-Pad2) -> VCC
- D173 pad 1: VCC -> Net-(D173-Pad1)
- D173 pad 2: Net-(D173-Pad2) -> GND
- D173 pad 3: GND -> Net-(D165-Pad1)
- D173 pad 4: Net-(D165-Pad2) -> VCC
- D174 pad 1: VCC -> Net-(D174-Pad1)
- D174 pad 2: Net-(D174-Pad2) -> GND
- D174 pad 3: GND -> Net-(D166-Pad1)
- D174 pad 4: Net-(D166-Pad2) -> VCC
- D175 pad 1: VCC -> Net-(D175-Pad1)
- D175 pad 2: Net-(D175-Pad2) -> GND
- D175 pad 3: GND -> Net-(D167-Pad1)
- D175 pad 4: Net-(D167-Pad2) -> VCC
- D176 pad 1: VCC -> Net-(D176-Pad1)
- D176 pad 2: Net-(D176-Pad2) -> GND
- D176 pad 3: GND -> Net-(D168-Pad1)
- D176 pad 4: Net-(D168-Pad2) -> VCC
- D177 pad 1: VCC -> Net-(D177-Pad1)
- D177 pad 2: Net-(D177-Pad2) -> GND
- D177 pad 3: GND -> Net-(D169-Pad1)
- D177 pad 4: Net-(D169-Pad2) -> VCC
- D178 pad 1: VCC -> Net-(D178-Pad1)
- D178 pad 2: Net-(D178-Pad2) -> GND
- D178 pad 3: GND -> Net-(D170-Pad1)
- D178 pad 4: Net-(D170-Pad2) -> VCC
- D179 pad 1: VCC -> Net-(D179-Pad1)
- D179 pad 2: Net-(D179-Pad2) -> GND
- D179 pad 3: GND -> Net-(D171-Pad1)
- D179 pad 4: Net-(D171-Pad2) -> VCC
- D180 pad 1: VCC -> Net-(D180-Pad1)
- D180 pad 2: Net-(D180-Pad2) -> GND
- D180 pad 3: GND -> Net-(D172-Pad1)
- D180 pad 4: Net-(D172-Pad2) -> VCC
- D181 pad 1: VCC -> Net-(D181-Pad1)
- D181 pad 2: Net-(D181-Pad2) -> GND
- D181 pad 3: GND -> Net-(D173-Pad1)
- D181 pad 4: Net-(D173-Pad2) -> VCC
- D182 pad 1: VCC -> Net-(D182-Pad1)
- D182 pad 2: Net-(D182-Pad2) -> GND
- D182 pad 3: GND -> Net-(D174-Pad1)
- D182 pad 4: Net-(D174-Pad2) -> VCC
- D183 pad 1: VCC -> Net-(D183-Pad1)
- D183 pad 2: Net-(D183-Pad2) -> GND
- D183 pad 3: GND -> Net-(D175-Pad1)
- D183 pad 4: Net-(D175-Pad2) -> VCC
- D184 pad 1: VCC -> Net-(D184-Pad1)
- D184 pad 2: Net-(D184-Pad2) -> GND
- D184 pad 3: GND -> Net-(D176-Pad1)
- D184 pad 4: Net-(D176-Pad2) -> VCC
- D185 pad 1: VCC -> Net-(D185-Pad1)
- D185 pad 2: Net-(D185-Pad2) -> GND
- D185 pad 3: GND -> Net-(D177-Pad1)
- D185 pad 4: Net-(D177-Pad2) -> VCC
- D186 pad 1: VCC -> Net-(D186-Pad1)
- D186 pad 2: Net-(D186-Pad2) -> GND
- D186 pad 3: GND -> Net-(D178-Pad1)
- D186 pad 4: Net-(D178-Pad2) -> VCC
- D187 pad 1: VCC -> Net-(D187-Pad1)
- D187 pad 2: Net-(D187-Pad2) -> GND
- D187 pad 3: GND -> Net-(D179-Pad1)
- D187 pad 4: Net-(D179-Pad2) -> VCC
- D188 pad 1: VCC -> Net-(D188-Pad1)
- D188 pad 2: Net-(D188-Pad2) -> GND
- D188 pad 3: GND -> Net-(D180-Pad1)
- D188 pad 4: Net-(D180-Pad2) -> VCC
- D189 pad 1: VCC -> Net-(D189-Pad1)
- D189 pad 2: Net-(D189-Pad2) -> GND
- D189 pad 3: GND -> Net-(D181-Pad1)
- D189 pad 4: Net-(D181-Pad2) -> VCC
- D190 pad 1: VCC -> Net-(D190-Pad1)
- D190 pad 2: Net-(D190-Pad2) -> GND
- D190 pad 3: GND -> Net-(D182-Pad1)
- D190 pad 4: Net-(D182-Pad2) -> VCC
- D191 pad 1: VCC -> Net-(D191-Pad1)
- D191 pad 2: Net-(D191-Pad2) -> GND
- D191 pad 3: GND -> Net-(D183-Pad1)
- D191 pad 4: Net-(D183-Pad2) -> VCC
- D192 pad 1: VCC -> Net-(D192-Pad1)
- D192 pad 2: Net-(D192-Pad2) -> GND
- D192 pad 3: GND -> Net-(D184-Pad1)
- D192 pad 4: Net-(D184-Pad2) -> VCC
- D193 pad 1: VCC -> Net-(D193-Pad1)
- D193 pad 2: Net-(D193-Pad2) -> GND
- D193 pad 3: GND -> Net-(D185-Pad1)
- D193 pad 4: Net-(D185-Pad2) -> VCC
- D194 pad 1: VCC -> Net-(D194-Pad1)
- D194 pad 2: Net-(D194-Pad2) -> GND
- D194 pad 3: GND -> Net-(D186-Pad1)
- D194 pad 4: Net-(D186-Pad2) -> VCC
- D195 pad 1: VCC -> Net-(D195-Pad1)
- D195 pad 2: Net-(D195-Pad2) -> GND
- D195 pad 3: GND -> Net-(D187-Pad1)
- D195 pad 4: Net-(D187-Pad2) -> VCC
- D196 pad 1: VCC -> Net-(D196-Pad1)
- D196 pad 2: Net-(D196-Pad2) -> GND
- D196 pad 3: GND -> Net-(D188-Pad1)
- D196 pad 4: Net-(D188-Pad2) -> VCC
- D197 pad 1: VCC -> Net-(D197-Pad1)
- D197 pad 2: Net-(D197-Pad2) -> GND
- D197 pad 3: GND -> Net-(D189-Pad1)
- D197 pad 4: Net-(D189-Pad2) -> VCC
- D198 pad 1: VCC -> Net-(D198-Pad1)
- D198 pad 2: Net-(D198-Pad2) -> GND
- D198 pad 3: GND -> Net-(D190-Pad1)
- D198 pad 4: Net-(D190-Pad2) -> VCC
- D199 pad 1: VCC -> Net-(D199-Pad1)
- D199 pad 2: Net-(D199-Pad2) -> GND
- D199 pad 3: GND -> Net-(D191-Pad1)
- D199 pad 4: Net-(D191-Pad2) -> VCC
- D200 pad 1: VCC -> Net-(D200-Pad1)
- D200 pad 2: Net-(D200-Pad2) -> GND
- D200 pad 3: GND -> Net-(D192-Pad1)
- D200 pad 4: Net-(D192-Pad2) -> VCC
- D201 pad 1: VCC -> Net-(D201-Pad1)
- D201 pad 2: Net-(D201-Pad2) -> GND
- D201 pad 3: GND -> Net-(D193-Pad1)
- D201 pad 4: Net-(D193-Pad2) -> VCC
- D202 pad 1: VCC -> Net-(D202-Pad1)
- D202 pad 2: Net-(D202-Pad2) -> GND
- D202 pad 3: GND -> Net-(D194-Pad1)
- D202 pad 4: Net-(D194-Pad2) -> VCC
- D203 pad 1: VCC -> Net-(D203-Pad1)
- D203 pad 2: Net-(D203-Pad2) -> GND
- D203 pad 3: GND -> Net-(D195-Pad1)
- D203 pad 4: Net-(D195-Pad2) -> VCC
- D204 pad 1: VCC -> Net-(D204-Pad1)
- D204 pad 2: Net-(D204-Pad2) -> GND
- D204 pad 3: GND -> Net-(D196-Pad1)
- D204 pad 4: Net-(D196-Pad2) -> VCC
- D205 pad 1: VCC -> Net-(D205-Pad1)
- D205 pad 2: Net-(D205-Pad2) -> GND
- D205 pad 3: GND -> Net-(D197-Pad1)
- D205 pad 4: Net-(D197-Pad2) -> VCC
- D206 pad 1: VCC -> Net-(D206-Pad1)
- D206 pad 2: Net-(D206-Pad2) -> GND
- D206 pad 3: GND -> Net-(D198-Pad1)
- D206 pad 4: Net-(D198-Pad2) -> VCC
- D207 pad 1: VCC -> Net-(D207-Pad1)
- D207 pad 2: Net-(D207-Pad2) -> GND
- D207 pad 3: GND -> Net-(D199-Pad1)
- D207 pad 4: Net-(D199-Pad2) -> VCC
- D208 pad 1: VCC -> Net-(D208-Pad1)
- D208 pad 2: Net-(D208-Pad2) -> GND
- D208 pad 3: GND -> Net-(D200-Pad1)
- D208 pad 4: Net-(D200-Pad2) -> VCC
- D209 pad 1: VCC -> Net-(D209-Pad1)
- D209 pad 2: Net-(D209-Pad2) -> GND
- D209 pad 3: GND -> Net-(D201-Pad1)
- D209 pad 4: Net-(D201-Pad2) -> VCC
- D210 pad 1: VCC -> Net-(D210-Pad1)
- D210 pad 2: Net-(D210-Pad2) -> GND
- D210 pad 3: GND -> Net-(D202-Pad1)
- D210 pad 4: Net-(D202-Pad2) -> VCC
- D211 pad 1: VCC -> Net-(D211-Pad1)
- D211 pad 2: Net-(D211-Pad2) -> GND
- D211 pad 3: GND -> Net-(D203-Pad1)
- D211 pad 4: Net-(D203-Pad2) -> VCC
- D212 pad 1: VCC -> Net-(D212-Pad1)
- D212 pad 2: Net-(D212-Pad2) -> GND
- D212 pad 3: GND -> Net-(D204-Pad1)
- D212 pad 4: Net-(D204-Pad2) -> VCC
- D213 pad 1: VCC -> Net-(D213-Pad1)
- D213 pad 2: Net-(D213-Pad2) -> GND
- D213 pad 3: GND -> Net-(D205-Pad1)
- D213 pad 4: Net-(D205-Pad2) -> VCC
- D214 pad 1: VCC -> Net-(D214-Pad1)
- D214 pad 2: Net-(D214-Pad2) -> GND
- D214 pad 3: GND -> Net-(D206-Pad1)
- D214 pad 4: Net-(D206-Pad2) -> VCC
- D215 pad 1: VCC -> Net-(D215-Pad1)
- D215 pad 2: Net-(D215-Pad2) -> GND
- D215 pad 3: GND -> Net-(D207-Pad1)
- D215 pad 4: Net-(D207-Pad2) -> VCC
- D216 pad 1: VCC -> Net-(D216-Pad1)
- D216 pad 2: Net-(D216-Pad2) -> GND
- D216 pad 3: GND -> Net-(D208-Pad1)
- D216 pad 4: Net-(D208-Pad2) -> VCC
- D217 pad 1: VCC -> Net-(D217-Pad1)
- D217 pad 2: Net-(D217-Pad2) -> GND
- D217 pad 3: GND -> Net-(D209-Pad1)
- D217 pad 4: Net-(D209-Pad2) -> VCC
- D218 pad 1: VCC -> Net-(D218-Pad1)
- D218 pad 2: Net-(D218-Pad2) -> GND
- D218 pad 3: GND -> Net-(D210-Pad1)
- D218 pad 4: Net-(D210-Pad2) -> VCC
- D219 pad 1: VCC -> Net-(D219-Pad1)
- D219 pad 2: Net-(D219-Pad2) -> GND
- D219 pad 3: GND -> Net-(D211-Pad1)
- D219 pad 4: Net-(D211-Pad2) -> VCC
- D220 pad 1: VCC -> Net-(D220-Pad1)
- D220 pad 2: Net-(D220-Pad2) -> GND
- D220 pad 3: GND -> Net-(D212-Pad1)
- D220 pad 4: Net-(D212-Pad2) -> VCC
- D221 pad 1: VCC -> Net-(D221-Pad1)
- D221 pad 2: Net-(D221-Pad2) -> GND
- D221 pad 3: GND -> Net-(D213-Pad1)
- D221 pad 4: Net-(D213-Pad2) -> VCC
- D222 pad 1: VCC -> Net-(D222-Pad1)
- D222 pad 2: Net-(D222-Pad2) -> GND
- D222 pad 3: GND -> Net-(D214-Pad1)
- D222 pad 4: Net-(D214-Pad2) -> VCC
- D223 pad 1: VCC -> Net-(D223-Pad1)
- D223 pad 2: Net-(D223-Pad2) -> GND
- D223 pad 3: GND -> Net-(D215-Pad1)
- D223 pad 4: Net-(D215-Pad2) -> VCC
- D224 pad 1: VCC -> Net-(D224-Pad1)
- D224 pad 2: Net-(D224-Pad2) -> GND
- D224 pad 3: GND -> Net-(D216-Pad1)
- D224 pad 4: Net-(D216-Pad2) -> VCC
- D225 pad 1: VCC -> Net-(D106-Pad3)
- D225 pad 2: Net-(D106-Pad4) -> GND
- D225 pad 3: GND -> Net-(D217-Pad1)
- D225 pad 4: Net-(D217-Pad2) -> VCC
- D226 pad 1: VCC -> Net-(D107-Pad3)
- D226 pad 2: Net-(D107-Pad4) -> GND
- D226 pad 3: GND -> Net-(D218-Pad1)
- D226 pad 4: Net-(D218-Pad2) -> VCC
- D227 pad 1: VCC -> Net-(D108-Pad3)
- D227 pad 2: Net-(D108-Pad4) -> GND
- D227 pad 3: GND -> Net-(D219-Pad1)
- D227 pad 4: Net-(D219-Pad2) -> VCC
- D228 pad 1: VCC -> Net-(D109-Pad3)
- D228 pad 2: Net-(D109-Pad4) -> GND
- D228 pad 3: GND -> Net-(D220-Pad1)
- D228 pad 4: Net-(D220-Pad2) -> VCC
- D229 pad 1: VCC -> Net-(D110-Pad3)
- D229 pad 2: Net-(D110-Pad4) -> GND
- D229 pad 3: GND -> Net-(D221-Pad1)
- D229 pad 4: Net-(D221-Pad2) -> VCC
- D230 pad 1: VCC -> Net-(D111-Pad3)
- D230 pad 2: Net-(D111-Pad4) -> GND
- D230 pad 3: GND -> Net-(D222-Pad1)
- D230 pad 4: Net-(D222-Pad2) -> VCC
- D231 pad 1: VCC -> Net-(D112-Pad3)
- D231 pad 2: Net-(D112-Pad4) -> GND
- D231 pad 3: GND -> Net-(D223-Pad1)
- D231 pad 4: Net-(D223-Pad2) -> VCC
- D232 pad 1: VCC -> Net-(D232-Pad1)
- D232 pad 2: Net-(D232-Pad2) -> GND
- D232 pad 3: GND -> Net-(D224-Pad1)
- D232 pad 4: Net-(D224-Pad2) -> VCC
