File: keyboard/keyboard.kicad_pcb (KiCad board)
At the start: 2 copper layers, 356 parts, among them K1 KEYSW, K10 KEYSW, K100 KEYSW, K101 KEYSW, K102 KEYSW, K103 KEYSW, K104 KEYSW, K11 KEYSW, K12 KEYSW, K13 KEYSW, K14 KEYSW, K15 KEYSW, K16 KEYSW, K17 KEYSW, K18 KEYSW, K19 KEYSW, K2 KEYSW, K20 KEYSW, K21 KEYSW, K22 KEYSW, K23 KEYSW, K24 KEYSW, K25 KEYSW, K26 KEYSW, K27 KEYSW, K28 KEYSW, K29 KEYSW, K3 KEYSW, K30 KEYSW, K31 KEYSW, K32 KEYSW, K33 KEYSW, K34 KEYSW, K35 KEYSW, K36 KEYSW, K37 KEYSW, K38 KEYSW, K39 KEYSW, K4 KEYSW, K40 KEYSW, K41 KEYSW, K42 KEYSW, K43 KEYSW, K44 KEYSW, K45 KEYSW, K46 KEYSW, K47 KEYSW, K48 KEYSW, K49 KEYSW, K5 KEYSW, K50 KEYSW, K51 KEYSW, K52 KEYSW, K53 KEYSW, K54 KEYSW, K55 KEYSW, K56 KEYSW, K57 KEYSW, K58 KEYSW, K59 KEYSW, K6 KEYSW, K60 KEYSW, K61 KEYSW, K62 KEYSW, K63 KEYSW, K64 KEYSW, K65 KEYSW, K66 KEYSW, K67 KEYSW, K68 KEYSW, K69 KEYSW, K7 KEYSW, K70 KEYSW, K71 KEYSW, K72 KEYSW, K73 KEYSW, K74 KEYSW, K75 KEYSW, K76 KEYSW, K77 KEYSW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

Commit message: arrange switches/diodes/other
Parts:
- added G***: LOGO, kbdlayout:keyboard_layout1, F.Cu at (209.0, 52.0)
- C3, C7, C8, D1, D10, D100, D101, D102, D103, D104, D11, D12, D13, D14, D15, D16, D17, D18, D19, D2, D20, D21, D22, D23, D24, D25, D26, D27, D28, D29, D3, D30, D31, D32, D33, D34, D35, D36, D37, D38, D39, D4, D40, D41, D42, D43, D44, D45, D46, D47, D48, D49, D5, D50, D51, D52, D53, D54, D55, D56, D58, D59, D6, D60, D61, D62, D63, D64, D65, D66, D67, D68, D7, D70, D71, D72, D73, D74, D75, D76, D77, D78, D79, D8, D80, D81, D82, D83, D85, D86, D87, D88, D89, D9, D90, D91, D92, D93, D94, D95, D98, D99, R1, R7, SW1, U1, X1: moved to B.Cu
- D105, D106, D107, D108, D109, D110, D111, D112, D113, D114, D115, D116, D117, D118, D119, D120, D121, D122, D123, D124, D125, D126, D127, D128, D129, D130, D131, D132, D133, D134, D135, D136, D137, D138, D139, D140, D141, D142, D143, D144, D145, D146, D147, D148, D149, D150, D151, D152, D153, D154, D155, D156, D157, D158, D159, D160, D161, D162, D163, D164, D165, D166, D167, D168, D169, D170, D171, D172, D173, D174, D175, D176, D177, D178, D179, D180, D181, D182, D183, D184, D185, D186, D187, D188, D189, D190, D191, D192, D193, D194, D195, D196, D197, D198, D199, D200, D201, D202, D203, D204, D205, D206, D207, D208, D209, D210, D211, D212, D213, D214, D215, D216, D217, D218, D219, D220, D221, D222, D223, D224, D225, D226, D227, D228, D229, D230, D231, D232: value WS2812B -> SK6812MINI; footprint LED_SMD:LED_WS2812B_PLCC4_5.0x5.0mm_P3.2mm -> LED_SMD:LED_SK6812MINI_PLCC4_3.5x3.5mm_P1.75mm; moved to B.Cu
- moved SW2 453.0 mm to (420.5, -13.5)
- moved C8 428.7 mm to (416.0, -0.50), turned to 90 degrees
- moved R6 413.3 mm to (420.5, -7.50), turned to 270 degrees
- moved R2 409.6 mm to (404.0, 1.50), turned to 270 degrees
- moved R4 406.9 mm to (408.5, -0.50), turned to 270 degrees
- moved R5 405.3 mm to (411.0, -0.50), turned to 270 degrees
- moved R3 404.1 mm to (402.0, 1.50), turned to 270 degrees
- moved D90 401.4 mm to (408.5, 28.5), turned to 270 degrees
- moved D95 398.0 mm to (418.0, 66.5)
- moved D98 396.2 mm to (408.5, 66.5), turned to 270 degrees
- moved D97 391.4 mm to (389.0, 66.5), turned to 90 degrees
- moved D94 386.9 mm to (408.5, 47.5), turned to 270 degrees
- moved C6 382.9 mm to (400.6, -9.40), turned to 90 degrees
- moved D115 381.6 mm to (565.0, 109.1)
- moved D157 380.6 mm to (549.3, 301.8)
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Connections:
- D105 pad 1: VCC -> Net-(D105-Pad1)
- D105 pad 2: Net-(D105-Pad2) -> GND
- D105 pad 3: GND -> /LEDDATA
- D105 pad 4: /LEDDATA -> VCC
- D106 pad 1: VCC -> Net-(D106-Pad1)
- D106 pad 2: Net-(D106-Pad2) -> GND
- D106 pad 3: GND -> Net-(D106-Pad3)
- D106 pad 4: Net-(D106-Pad4) -> VCC
- D107 pad 1: VCC -> Net-(D107-Pad1)
- D107 pad 2: Net-(D107-Pad2) -> GND
- D107 pad 3: GND -> Net-(D107-Pad3)
- D107 pad 4: Net-(D107-Pad4) -> VCC
- D108 pad 1: VCC -> Net-(D108-Pad1)
- D108 pad 2: Net-(D108-Pad2) -> GND
- D108 pad 3: GND -> Net-(D108-Pad3)
- D108 pad 4: Net-(D108-Pad4) -> VCC
- D109 pad 1: VCC -> Net-(D109-Pad1)
- D109 pad 2: Net-(D109-Pad2) -> GND
- D109 pad 3: GND -> Net-(D109-Pad3)
- D109 pad 4: Net-(D109-Pad4) -> VCC
- D110 pad 1: VCC -> Net-(D110-Pad1)
- D110 pad 2: Net-(D110-Pad2) -> GND
- D110 pad 3: GND -> Net-(D110-Pad3)
- D110 pad 4: Net-(D110-Pad4) -> VCC
- D111 pad 1: VCC -> Net-(D111-Pad1)
- D111 pad 2: Net-(D111-Pad2) -> GND
- D111 pad 3: GND -> Net-(D111-Pad3)
- D111 pad 4: Net-(D111-Pad4) -> VCC
- D112 pad 1: VCC -> Net-(D112-Pad1)
- D112 pad 2: Net-(D112-Pad2) -> GND
- D112 pad 3: GND -> Net-(D112-Pad3)
- D112 pad 4: Net-(D112-Pad4) -> VCC
- D113 pad 1: VCC -> Net-(D113-Pad1)
- D113 pad 2: Net-(D113-Pad2) -> GND
- D113 pad 3: GND -> Net-(D105-Pad1)
- D113 pad 4: Net-(D105-Pad2) -> VCC
- D114 pad 1: VCC -> Net-(D114-Pad1)
- D114 pad 2: Net-(D114-Pad2) -> GND
- D114 pad 3: GND -> Net-(D106-Pad1)
- D114 pad 4: Net-(D106-Pad2) -> VCC
- D115 pad 1: VCC -> Net-(D115-Pad1)
- D115 pad 2: Net-(D115-Pad2) -> GND
- D115 pad 3: GND -> Net-(D107-Pad1)
- D115 pad 4: Net-(D107-Pad2) -> VCC
- D116 pad 1: VCC -> Net-(D116-Pad1)
- D116 pad 2: Net-(D116-Pad2) -> GND
- D116 pad 3: GND -> Net-(D108-Pad1)
- D116 pad 4: Net-(D108-Pad2) -> VCC
- D117 pad 1: VCC -> Net-(D117-Pad1)
- D117 pad 2: Net-(D117-Pad2) -> GND
- D117 pad 3: GND -> Net-(D109-Pad1)
- D117 pad 4: Net-(D109-Pad2) -> VCC
- D118 pad 1: VCC -> Net-(D118-Pad1)
- D118 pad 2: Net-(D118-Pad2) -> GND
- D118 pad 3: GND -> Net-(D110-Pad1)
- D118 pad 4: Net-(D110-Pad2) -> VCC
- D119 pad 1: VCC -> Net-(D119-Pad1)
- D119 pad 2: Net-(D119-Pad2) -> GND
- D119 pad 3: GND -> Net-(D111-Pad1)
- D119 pad 4: Net-(D111-Pad2) -> VCC
- D120 pad 1: VCC -> Net-(D120-Pad1)
- D120 pad 2: Net-(D120-Pad2) -> GND
- D120 pad 3: GND -> Net-(D112-Pad1)
- D120 pad 4: Net-(D112-Pad2) -> VCC
- D121 pad 1: VCC -> Net-(D121-Pad1)
- D121 pad 2: Net-(D121-Pad2) -> GND
- D121 pad 3: GND -> Net-(D113-Pad1)
- D121 pad 4: Net-(D113-Pad2) -> VCC
- D122 pad 1: VCC -> Net-(D122-Pad1)
- D122 pad 2: Net-(D122-Pad2) -> GND
- D122 pad 3: GND -> Net-(D114-Pad1)
- D122 pad 4: Net-(D114-Pad2) -> VCC
- D123 pad 1: VCC -> Net-(D123-Pad1)
- D123 pad 2: Net-(D123-Pad2) -> GND
- D123 pad 3: GND -> Net-(D115-Pad1)
- D123 pad 4: Net-(D115-Pad2) -> VCC
- D124 pad 1: VCC -> Net-(D124-Pad1)
- D124 pad 2: Net-(D124-Pad2) -> GND
- D124 pad 3: GND -> Net-(D116-Pad1)
- D124 pad 4: Net-(D116-Pad2) -> VCC
- D125 pad 1: VCC -> Net-(D125-Pad1)
- D125 pad 2: Net-(D125-Pad2) -> GND
- D125 pad 3: GND -> Net-(D117-Pad1)
- D125 pad 4: Net-(D117-Pad2) -> VCC
- D126 pad 1: VCC -> Net-(D126-Pad1)
- D126 pad 2: Net-(D126-Pad2) -> GND
- D126 pad 3: GND -> Net-(D118-Pad1)
- D126 pad 4: Net-(D118-Pad2) -> VCC
- D127 pad 1: VCC -> Net-(D127-Pad1)
- D127 pad 2: Net-(D127-Pad2) -> GND
- D127 pad 3: GND -> Net-(D119-Pad1)
- D127 pad 4: Net-(D119-Pad2) -> VCC
- D128 pad 1: VCC -> Net-(D128-Pad1)
- D128 pad 2: Net-(D128-Pad2) -> GND
- D128 pad 3: GND -> Net-(D120-Pad1)
- D128 pad 4: Net-(D120-Pad2) -> VCC
- D129 pad 1: VCC -> Net-(D129-Pad1)
- D129 pad 2: Net-(D129-Pad2) -> GND
- D129 pad 3: GND -> Net-(D121-Pad1)
- D129 pad 4: Net-(D121-Pad2) -> VCC
- D130 pad 1: VCC -> Net-(D130-Pad1)
- D130 pad 2: Net-(D130-Pad2) -> GND
- D130 pad 3: GND -> Net-(D122-Pad1)
- D130 pad 4: Net-(D122-Pad2) -> VCC
- D131 pad 1: VCC -> Net-(D131-Pad1)
- D131 pad 2: Net-(D131-Pad2) -> GND
- D131 pad 3: GND -> Net-(D123-Pad1)
- D131 pad 4: Net-(D123-Pad2) -> VCC
- D132 pad 1: VCC -> Net-(D132-Pad1)
- D132 pad 2: Net-(D132-Pad2) -> GND
- D132 pad 3: GND -> Net-(D124-Pad1)
- D132 pad 4: Net-(D124-Pad2) -> VCC
- D133 pad 1: VCC -> Net-(D133-Pad1)
- D133 pad 2: Net-(D133-Pad2) -> GND
- D133 pad 3: GND -> Net-(D125-Pad1)
- D133 pad 4: Net-(D125-Pad2) -> VCC
- D134 pad 1: VCC -> Net-(D134-Pad1)
- D134 pad 2: Net-(D134-Pad2) -> GND
- D134 pad 3: GND -> Net-(D126-Pad1)
- D134 pad 4: Net-(D126-Pad2) -> VCC
- D135 pad 1: VCC -> Net-(D135-Pad1)
- D135 pad 2: Net-(D135-Pad2) -> GND
- D135 pad 3: GND -> Net-(D127-Pad1)
- D135 pad 4: Net-(D127-Pad2) -> VCC
- D136 pad 1: VCC -> Net-(D136-Pad1)
- D136 pad 2: Net-(D136-Pad2) -> GND
- D136 pad 3: GND -> Net-(D128-Pad1)
- D136 pad 4: Net-(D128-Pad2) -> VCC
- D137 pad 1: VCC -> Net-(D137-Pad1)
- D137 pad 2: Net-(D137-Pad2) -> GND
- D137 pad 3: GND -> Net-(D129-Pad1)
- D137 pad 4: Net-(D129-Pad2) -> VCC
- D138 pad 1: VCC -> Net-(D138-Pad1)
- D138 pad 2: Net-(D138-Pad2) -> GND
- D138 pad 3: GND -> Net-(D130-Pad1)
- D138 pad 4: Net-(D130-Pad2) -> VCC
- D139 pad 1: VCC -> Net-(D139-Pad1)
- D139 pad 2: Net-(D139-Pad2) -> GND
- D139 pad 3: GND -> Net-(D131-Pad1)
- D139 pad 4: Net-(D131-Pad2) -> VCC
- D140 pad 1: VCC -> Net-(D140-Pad1)
- D140 pad 2: Net-(D140-Pad2) -> GND
- D140 pad 3: GND -> Net-(D132-Pad1)
- D140 pad 4: Net-(D132-Pad2) -> VCC
- D141 pad 1: VCC -> Net-(D141-Pad1)
- D141 pad 2: Net-(D141-Pad2) -> GND
- D141 pad 3: GND -> Net-(D133-Pad1)
- D141 pad 4: Net-(D133-Pad2) -> VCC
- D142 pad 1: VCC -> Net-(D142-Pad1)
- D142 pad 2: Net-(D142-Pad2) -> GND
- D142 pad 3: GND -> Net-(D134-Pad1)
- D142 pad 4: Net-(D134-Pad2) -> VCC
- D143 pad 1: VCC -> Net-(D143-Pad1)
- D143 pad 2: Net-(D143-Pad2) -> GND
- D143 pad 3: GND -> Net-(D135-Pad1)
- D143 pad 4: Net-(D135-Pad2) -> VCC
- D144 pad 1: VCC -> Net-(D144-Pad1)
- D144 pad 2: Net-(D144-Pad2) -> GND
- D144 pad 3: GND -> Net-(D136-Pad1)
- D144 pad 4: Net-(D136-Pad2) -> VCC
- D145 pad 1: VCC -> Net-(D145-Pad1)
- D145 pad 2: Net-(D145-Pad2) -> GND
- D145 pad 3: GND -> Net-(D137-Pad1)
- D145 pad 4: Net-(D137-Pad2) -> VCC
- D146 pad 1: VCC -> Net-(D146-Pad1)
- D146 pad 2: Net-(D146-Pad2) -> GND
- D146 pad 3: GND -> Net-(D138-Pad1)
- D146 pad 4: Net-(D138-Pad2) -> VCC
- D147 pad 1: VCC -> Net-(D147-Pad1)
- D147 pad 2: Net-(D147-Pad2) -> GND
- D147 pad 3: GND -> Net-(D139-Pad1)
- D147 pad 4: Net-(D139-Pad2) -> VCC
- D148 pad 1: VCC -> Net-(D148-Pad1)
- D148 pad 2: Net-(D148-Pad2) -> GND
- D148 pad 3: GND -> Net-(D140-Pad1)
- D148 pad 4: Net-(D140-Pad2) -> VCC
- D149 pad 1: VCC -> Net-(D149-Pad1)
- D149 pad 2: Net-(D149-Pad2) -> GND
- D149 pad 3: GND -> Net-(D141-Pad1)
- D149 pad 4: Net-(D141-Pad2) -> VCC
- D150 pad 1: VCC -> Net-(D150-Pad1)
- D150 pad 2: Net-(D150-Pad2) -> GND
- D150 pad 3: GND -> Net-(D142-Pad1)
- D150 pad 4: Net-(D142-Pad2) -> VCC
- D151 pad 1: VCC -> Net-(D151-Pad1)
- D151 pad 2: Net-(D151-Pad2) -> GND
- D151 pad 3: GND -> Net-(D143-Pad1)
- D151 pad 4: Net-(D143-Pad2) -> VCC
- D152 pad 1: VCC -> Net-(D152-Pad1)
- D152 pad 2: Net-(D152-Pad2) -> GND
- D152 pad 3: GND -> Net-(D144-Pad1)
- D152 pad 4: Net-(D144-Pad2) -> VCC
- D153 pad 1: VCC -> Net-(D153-Pad1)
- D153 pad 2: Net-(D153-Pad2) -> GND
- D153 pad 3: GND -> Net-(D145-Pad1)
- D153 pad 4: Net-(D145-Pad2) -> VCC
- D154 pad 1: VCC -> Net-(D154-Pad1)
- D154 pad 2: Net-(D154-Pad2) -> GND
- D154 pad 3: GND -> Net-(D146-Pad1)
- D154 pad 4: Net-(D146-Pad2) -> VCC
- D155 pad 1: VCC -> Net-(D155-Pad1)
- D155 pad 2: Net-(D155-Pad2) -> GND
- D155 pad 3: GND -> Net-(D147-Pad1)
- D155 pad 4: Net-(D147-Pad2) -> VCC
- D156 pad 1: VCC -> Net-(D156-Pad1)
- D156 pad 2: Net-(D156-Pad2) -> GND
- D156 pad 3: GND -> Net-(D148-Pad1)
- D156 pad 4: Net-(D148-Pad2) -> VCC
- D157 pad 1: VCC -> Net-(D157-Pad1)
- D157 pad 2: Net-(D157-Pad2) -> GND
- D157 pad 3: GND -> Net-(D149-Pad1)
- D157 pad 4: Net-(D149-Pad2) -> VCC
- D158 pad 1: VCC -> Net-(D158-Pad1)
- D158 pad 2: Net-(D158-Pad2) -> GND
- D158 pad 3: GND -> Net-(D150-Pad1)
- D158 pad 4: Net-(D150-Pad2) -> VCC
- D159 pad 1: VCC -> Net-(D159-Pad1)
- D159 pad 2: Net-(D159-Pad2) -> GND
- D159 pad 3: GND -> Net-(D151-Pad1)
- D159 pad 4: Net-(D151-Pad2) -> VCC
- D160 pad 1: VCC -> Net-(D160-Pad1)
- D160 pad 2: Net-(D160-Pad2) -> GND
- D160 pad 3: GND -> Net-(D152-Pad1)
- D160 pad 4: Net-(D152-Pad2) -> VCC
- D161 pad 1: VCC -> Net-(D161-Pad1)
- D161 pad 2: Net-(D161-Pad2) -> GND
- D161 pad 3: GND -> Net-(D153-Pad1)
- D161 pad 4: Net-(D153-Pad2) -> VCC
- D162 pad 1: VCC -> Net-(D162-Pad1)
- D162 pad 2: Net-(D162-Pad2) -> GND
- D162 pad 3: GND -> Net-(D154-Pad1)
- D162 pad 4: Net-(D154-Pad2) -> VCC
- D163 pad 1: VCC -> Net-(D163-Pad1)
- D163 pad 2: Net-(D163-Pad2) -> GND
- D163 pad 3: GND -> Net-(D155-Pad1)
- D163 pad 4: Net-(D155-Pad2) -> VCC
- D164 pad 1: VCC -> Net-(D164-Pad1)
- D164 pad 2: Net-(D164-Pad2) -> GND
- D164 pad 3: GND -> Net-(D156-Pad1)
- D164 pad 4: Net-(D156-Pad2) -> VCC
- D165 pad 1: VCC -> Net-(D165-Pad1)
- D165 pad 2: Net-(D165-Pad2) -> GND
- D165 pad 3: GND -> Net-(D157-Pad1)
- D165 pad 4: Net-(D157-Pad2) -> VCC
- D166 pad 1: VCC -> Net-(D166-Pad1)
- D166 pad 2: Net-(D166-Pad2) -> GND
- D166 pad 3: GND -> Net-(D158-Pad1)
- D166 pad 4: Net-(D158-Pad2) -> VCC
- D167 pad 1: VCC -> Net-(D167-Pad1)
- D167 pad 2: Net-(D167-Pad2) -> GND
- D167 pad 3: GND -> Net-(D159-Pad1)
- D167 pad 4: Net-(D159-Pad2) -> VCC
- D168 pad 1: VCC -> Net-(D168-Pad1)
- D168 pad 2: Net-(D168-Pad2) -> GND
- D168 pad 3: GND -> Net-(D160-Pad1)
- D168 pad 4: Net-(D160-Pad2) -> VCC
- D169 pad 1: VCC -> Net-(D169-Pad1)
- D169 pad 2: Net-(D169-Pad2) -> GND
- D169 pad 3: GND -> Net-(D161-Pad1)
- D169 pad 4: Net-(D161-Pad2) -> VCC
- D170 pad 1: VCC -> Net-(D170-Pad1)
- D170 pad 2: Net-(D170-Pad2) -> GND
- D170 pad 3: GND -> Net-(D162-Pad1)
- D170 pad 4: Net-(D162-Pad2) -> VCC
- D171 pad 1: VCC -> Net-(D171-Pad1)
- D171 pad 2: Net-(D171-Pad2) -> GND
- D171 pad 3: GND -> Net-(D163-Pad1)
- D171 pad 4: Net-(D163-Pad2) -> VCC
- D172 pad 1: VCC -> Net-(D172-Pad1)
- D172 pad 2: Net-(D172-Pad2) -> GND
- D172 pad 3: GND -> Net-(D164-Pad1)
- D172 pad 4: Net-(D164-Pad2) -> VCC
- D173 pad 1: VCC -> Net-(D173-Pad1)
- D173 pad 2: Net-(D173-Pad2) -> GND
- D173 pad 3: GND -> Net-(D165-Pad1)
- D173 pad 4: Net-(D165-Pad2) -> VCC
- D174 pad 1: VCC -> Net-(D174-Pad1)
- D174 pad 2: Net-(D174-Pad2) -> GND
- D174 pad 3: GND -> Net-(D166-Pad1)
- D174 pad 4: Net-(D166-Pad2) -> VCC
- D175 pad 1: VCC -> Net-(D175-Pad1)
- D175 pad 2: Net-(D175-Pad2) -> GND
- D175 pad 3: GND -> Net-(D167-Pad1)
- D175 pad 4: Net-(D167-Pad2) -> VCC
- D176 pad 1: VCC -> Net-(D176-Pad1)
- D176 pad 2: Net-(D176-Pad2) -> GND
- D176 pad 3: GND -> Net-(D168-Pad1)
- D176 pad 4: Net-(D168-Pad2) -> VCC
- D177 pad 1: VCC -> Net-(D177-Pad1)
- D177 pad 2: Net-(D177-Pad2) -> GND
- D177 pad 3: GND -> Net-(D169-Pad1)
- D177 pad 4: Net-(D169-Pad2) -> VCC
- D178 pad 1: VCC -> Net-(D178-Pad1)
- D178 pad 2: Net-(D178-Pad2) -> GND
- D178 pad 3: GND -> Net-(D170-Pad1)
- D178 pad 4: Net-(D170-Pad2) -> VCC
- D179 pad 1: VCC -> Net-(D179-Pad1)
- D179 pad 2: Net-(D179-Pad2) -> GND
- D179 pad 3: GND -> Net-(D171-Pad1)
- D179 pad 4: Net-(D171-Pad2) -> VCC
- D180 pad 1: VCC -> Net-(D180-Pad1)
- D180 pad 2: Net-(D180-Pad2) -> GND
- D180 pad 3: GND -> Net-(D172-Pad1)
- D180 pad 4: Net-(D172-Pad2) -> VCC
- D181 pad 1: VCC -> Net-(D181-Pad1)
- D181 pad 2: Net-(D181-Pad2) -> GND
- D181 pad 3: GND -> Net-(D173-Pad1)
- D181 pad 4: Net-(D173-Pad2) -> VCC
- D182 pad 1: VCC -> Net-(D182-Pad1)
- D182 pad 2: Net-(D182-Pad2) -> GND
- D182 pad 3: GND -> Net-(D174-Pad1)
- D182 pad 4: Net-(D174-Pad2) -> VCC
- D183 pad 1: VCC -> Net-(D183-Pad1)
- D183 pad 2: Net-(D183-Pad2) -> GND
- D183 pad 3: GND -> Net-(D175-Pad1)
- D183 pad 4: Net-(D175-Pad2) -> VCC
- D184 pad 1: VCC -> Net-(D184-Pad1)
- D184 pad 2: Net-(D184-Pad2) -> GND
- D184 pad 3: GND -> Net-(D176-Pad1)
- D184 pad 4: Net-(D176-Pad2) -> VCC
- D185 pad 1: VCC -> Net-(D185-Pad1)
- D185 pad 2: Net-(D185-Pad2) -> GND
- D185 pad 3: GND -> Net-(D177-Pad1)
- D185 pad 4: Net-(D177-Pad2) -> VCC
- D186 pad 1: VCC -> Net-(D186-Pad1)
- D186 pad 2: Net-(D186-Pad2) -> GND
- D186 pad 3: GND -> Net-(D178-Pad1)
- D186 pad 4: Net-(D178-Pad2) -> VCC
- D187 pad 1: VCC -> Net-(D187-Pad1)
- D187 pad 2: Net-(D187-Pad2) -> GND
- D187 pad 3: GND -> Net-(D179-Pad1)
- D187 pad 4: Net-(D179-Pad2) -> VCC
- D188 pad 1: VCC -> Net-(D188-Pad1)
- D188 pad 2: Net-(D188-Pad2) -> GND
- D188 pad 3: GND -> Net-(D180-Pad1)
- D188 pad 4: Net-(D180-Pad2) -> VCC
- D189 pad 1: VCC -> Net-(D189-Pad1)
- D189 pad 2: Net-(D189-Pad2) -> GND
- D189 pad 3: GND -> Net-(D181-Pad1)
- D189 pad 4: Net-(D181-Pad2) -> VCC
- D190 pad 1: VCC -> Net-(D190-Pad1)
- D190 pad 2: Net-(D190-Pad2) -> GND
- D190 pad 3: GND -> Net-(D182-Pad1)
- D190 pad 4: Net-(D182-Pad2) -> VCC
- D191 pad 1: VCC -> Net-(D191-Pad1)
- D191 pad 2: Net-(D191-Pad2) -> GND
- D191 pad 3: GND -> Net-(D183-Pad1)
- D191 pad 4: Net-(D183-Pad2) -> VCC
- D192 pad 1: VCC -> Net-(D192-Pad1)
- D192 pad 2: Net-(D192-Pad2) -> GND
- D192 pad 3: GND -> Net-(D184-Pad1)
- D192 pad 4: Net-(D184-Pad2) -> VCC
- D193 pad 1: VCC -> Net-(D193-Pad1)
- D193 pad 2: Net-(D193-Pad2) -> GND
- D193 pad 3: GND -> Net-(D185-Pad1)
- D193 pad 4: Net-(D185-Pad2) -> VCC
- D194 pad 1: VCC -> Net-(D194-Pad1)
- D194 pad 2: Net-(D194-Pad2) -> GND
- D194 pad 3: GND -> Net-(D186-Pad1)
- D194 pad 4: Net-(D186-Pad2) -> VCC
- D195 pad 1: VCC -> Net-(D195-Pad1)
- D195 pad 2: Net-(D195-Pad2) -> GND
- D195 pad 3: GND -> Net-(D187-Pad1)
- D195 pad 4: Net-(D187-Pad2) -> VCC
- D196 pad 1: VCC -> Net-(D196-Pad1)
- D196 pad 2: Net-(D196-Pad2) -> GND
- D196 pad 3: GND -> Net-(D188-Pad1)
- D196 pad 4: Net-(D188-Pad2) -> VCC
- D197 pad 1: VCC -> Net-(D197-Pad1)
- D197 pad 2: Net-(D197-Pad2) -> GND
- D197 pad 3: GND -> Net-(D189-Pad1)
- D197 pad 4: Net-(D189-Pad2) -> VCC
- D198 pad 1: VCC -> Net-(D198-Pad1)
- D198 pad 2: Net-(D198-Pad2) -> GND
- D198 pad 3: GND -> Net-(D190-Pad1)
- D198 pad 4: Net-(D190-Pad2) -> VCC
- D199 pad 1: VCC -> Net-(D199-Pad1)
- D199 pad 2: Net-(D199-Pad2) -> GND
- D199 pad 3: GND -> Net-(D191-Pad1)
- D199 pad 4: Net-(D191-Pad2) -> VCC
- D200 pad 1: VCC -> Net-(D200-Pad1)
- D200 pad 2: Net-(D200-Pad2) -> GND
- D200 pad 3: GND -> Net-(D192-Pad1)
- D200 pad 4: Net-(D192-Pad2) -> VCC
- D201 pad 1: VCC -> Net-(D201-Pad1)
- D201 pad 2: Net-(D201-Pad2) -> GND
- D201 pad 3: GND -> Net-(D193-Pad1)
- D201 pad 4: Net-(D193-Pad2) -> VCC
- D202 pad 1: VCC -> Net-(D202-Pad1)
- D202 pad 2: Net-(D202-Pad2) -> GND
- D202 pad 3: GND -> Net-(D194-Pad1)
- D202 pad 4: Net-(D194-Pad2) -> VCC
- D203 pad 1: VCC -> Net-(D203-Pad1)
- D203 pad 2: Net-(D203-Pad2) -> GND
- D203 pad 3: GND -> Net-(D195-Pad1)
- D203 pad 4: Net-(D195-Pad2) -> VCC
- D204 pad 1: VCC -> Net-(D204-Pad1)
- D204 pad 2: Net-(D204-Pad2) -> GND
- D204 pad 3: GND -> Net-(D196-Pad1)
- D204 pad 4: Net-(D196-Pad2) -> VCC
- D205 pad 1: VCC -> Net-(D205-Pad1)
- D205 pad 2: Net-(D205-Pad2) -> GND
- D205 pad 3: GND -> Net-(D197-Pad1)
- D205 pad 4: Net-(D197-Pad2) -> VCC
- D206 pad 1: VCC -> Net-(D206-Pad1)
- D206 pad 2: Net-(D206-Pad2) -> GND
- D206 pad 3: GND -> Net-(D198-Pad1)
- D206 pad 4: Net-(D198-Pad2) -> VCC
- D207 pad 1: VCC -> Net-(D207-Pad1)
- D207 pad 2: Net-(D207-Pad2) -> GND
- D207 pad 3: GND -> Net-(D199-Pad1)
- D207 pad 4: Net-(D199-Pad2) -> VCC
- D208 pad 1: VCC -> Net-(D208-Pad1)
- D208 pad 2: Net-(D208-Pad2) -> GND
- D208 pad 3: GND -> Net-(D200-Pad1)
- D208 pad 4: Net-(D200-Pad2) -> VCC
- D209 pad 1: VCC -> Net-(D209-Pad1)
- D209 pad 2: Net-(D209-Pad2) -> GND
- D209 pad 3: GND -> Net-(D201-Pad1)
- D209 pad 4: Net-(D201-Pad2) -> VCC
- D210 pad 1: VCC -> Net-(D210-Pad1)
- D210 pad 2: Net-(D210-Pad2) -> GND
- D210 pad 3: GND -> Net-(D202-Pad1)
- D210 pad 4: Net-(D202-Pad2) -> VCC
- D211 pad 1: VCC -> Net-(D211-Pad1)
- D211 pad 2: Net-(D211-Pad2) -> GND
- D211 pad 3: GND -> Net-(D203-Pad1)
- D211 pad 4: Net-(D203-Pad2) -> VCC
- D212 pad 1: VCC -> Net-(D212-Pad1)
- D212 pad 2: Net-(D212-Pad2) -> GND
- D212 pad 3: GND -> Net-(D204-Pad1)
- D212 pad 4: Net-(D204-Pad2) -> VCC
- D213 pad 1: VCC -> Net-(D213-Pad1)
- D213 pad 2: Net-(D213-Pad2) -> GND
- D213 pad 3: GND -> Net-(D205-Pad1)
- D213 pad 4: Net-(D205-Pad2) -> VCC
- D214 pad 1: VCC -> Net-(D214-Pad1)
- D214 pad 2: Net-(D214-Pad2) -> GND
- D214 pad 3: GND -> Net-(D206-Pad1)
- D214 pad 4: Net-(D206-Pad2) -> VCC
- D215 pad 1: VCC -> Net-(D215-Pad1)
- D215 pad 2: Net-(D215-Pad2) -> GND
- D215 pad 3: GND -> Net-(D207-Pad1)
- D215 pad 4: Net-(D207-Pad2) -> VCC
- D216 pad 1: VCC -> Net-(D216-Pad1)
- D216 pad 2: Net-(D216-Pad2) -> GND
- D216 pad 3: GND -> Net-(D208-Pad1)
- D216 pad 4: Net-(D208-Pad2) -> VCC
- D217 pad 1: VCC -> Net-(D217-Pad1)
- D217 pad 2: Net-(D217-Pad2) -> GND
- D217 pad 3: GND -> Net-(D209-Pad1)
- D217 pad 4: Net-(D209-Pad2) -> VCC
- D218 pad 1: VCC -> Net-(D218-Pad1)
- D218 pad 2: Net-(D218-Pad2) -> GND
- D218 pad 3: GND -> Net-(D210-Pad1)
- D218 pad 4: Net-(D210-Pad2) -> VCC
- D219 pad 1: VCC -> Net-(D219-Pad1)
- D219 pad 2: Net-(D219-Pad2) -> GND
- D219 pad 3: GND -> Net-(D211-Pad1)
- D219 pad 4: Net-(D211-Pad2) -> VCC
- D220 pad 1: VCC -> Net-(D220-Pad1)
- D220 pad 2: Net-(D220-Pad2) -> GND
- D220 pad 3: GND -> Net-(D212-Pad1)
- D220 pad 4: Net-(D212-Pad2) -> VCC
- D221 pad 1: VCC -> Net-(D221-Pad1)
- D221 pad 2: Net-(D221-Pad2) -> GND
- D221 pad 3: GND -> Net-(D213-Pad1)
- D221 pad 4: Net-(D213-Pad2) -> VCC
- D222 pad 1: VCC -> Net-(D222-Pad1)
- D222 pad 2: Net-(D222-Pad2) -> GND
- D222 pad 3: GND -> Net-(D214-Pad1)
- D222 pad 4: Net-(D214-Pad2) -> VCC
- D223 pad 1: VCC -> Net-(D223-Pad1)
- D223 pad 2: Net-(D223-Pad2) -> GND
- D223 pad 3: GND -> Net-(D215-Pad1)
- D223 pad 4: Net-(D215-Pad2) -> VCC
- D224 pad 1: VCC -> Net-(D224-Pad1)
- D224 pad 2: Net-(D224-Pad2) -> GND
- D224 pad 3: GND -> Net-(D216-Pad1)
- D224 pad 4: Net-(D216-Pad2) -> VCC
- D225 pad 1: VCC -> Net-(D106-Pad3)
- D225 pad 2: Net-(D106-Pad4) -> GND
- D225 pad 3: GND -> Net-(D217-Pad1)
- D225 pad 4: Net-(D217-Pad2) -> VCC
- D226 pad 1: VCC -> Net-(D107-Pad3)
- D226 pad 2: Net-(D107-Pad4) -> GND
- D226 pad 3: GND -> Net-(D218-Pad1)
- D226 pad 4: Net-(D218-Pad2) -> VCC
- D227 pad 1: VCC -> Net-(D108-Pad3)
- D227 pad 2: Net-(D108-Pad4) -> GND
- D227 pad 3: GND -> Net-(D219-Pad1)
- D227 pad 4: Net-(D219-Pad2) -> VCC
- D228 pad 1: VCC -> Net-(D109-Pad3)
- D228 pad 2: Net-(D109-Pad4) -> GND
- D228 pad 3: GND -> Net-(D220-Pad1)
- D228 pad 4: Net-(D220-Pad2) -> VCC
- D229 pad 1: VCC -> Net-(D110-Pad3)
- D229 pad 2: Net-(D110-Pad4) -> GND
- D229 pad 3: GND -> Net-(D221-Pad1)
- D229 pad 4: Net-(D221-Pad2) -> VCC
- D230 pad 1: VCC -> Net-(D111-Pad3)
- D230 pad 2: Net-(D111-Pad4) -> GND
- D230 pad 3: GND -> Net-(D222-Pad1)
- D230 pad 4: Net-(D222-Pad2) -> VCC
- D231 pad 1: VCC -> Net-(D112-Pad3)
- D231 pad 2: Net-(D112-Pad4) -> GND
- D231 pad 3: GND -> Net-(D223-Pad1)
- D231 pad 4: Net-(D223-Pad2) -> VCC
- D232 pad 1: VCC -> Net-(D232-Pad1)
- D232 pad 2: Net-(D232-Pad2) -> GND
- D232 pad 3: GND -> Net-(D224-Pad1)
- D232 pad 4: Net-(D224-Pad2) -> VCC
- U1 pad 16: Net-(C3-Pad1) -> Net-(C7-Pad1)
- U1 pad 17: Net-(C7-Pad1) -> Net-(C3-Pad1)
- U1 pad 27: /col12 -> /col1
- U1 pad 28: /col11 -> /col2
- U1 pad 29: /col10 -> /col3
- U1 pad 30: /col9 -> /col4
- U1 pad 31: /col8 -> /col5
- U1 pad 32: /col7 -> /col6
- U1 pad 36: /col6 -> /col7
- U1 pad 37: /col5 -> /col8
- U1 pad 38: /col4 -> /col9
- U1 pad 39: /col3 -> /col10
- U1 pad 40: /col2 -> /col11
- U1 pad 41: /col1 -> /col12

Commit message: finally figure out leds & remove led drivers
Parts:
- removed C3: 22p, Capacitor_SMD:C_0805_2012Metric
- removed the C7 at (364.9, 5.80)
- removed C8: 1u, Capacitor_SMD:C_0805_2012Metric
- removed D105, D106, D107, D108, D109, D110, D111, D112, D113, D114, D115, D116, D117, D118, D119, D120, D121, D122, D123, D124, D125, D126, D127, D128, D129, D130, D131, D132, D133, D134, D135, D136, D137, D138, D139, D140, D141, D142, D143, D144, D145, D146, D147, D148, D149, D150, D151, D152, D153, D154, D155, D156, D157, D158, D159, D160, D161, D162, D163, D164, D165, D166, D167, D168, D169, D170, D171, D172, D173, D174, D175, D176, D177, D178, D179, D180, D181, D182, D183, D184, D185, D186, D187, D188, D189, D190, D191, D192, D193, D194, D195, D196, D197, D198, D199, D200, D201, D202, D203, D204, D205, D206, D207, D208, D209, D210, D211, D212, D213, D214, D215, D216, D217, D218, D219, D220, D221, D222, D223, D224, D225, D226, D227, D228, D229, D230, D231, D232: SK6812MINI, LED_SMD:LED_SK6812MINI_PLCC4_3.5x3.5mm_P1.75mm
- removed X1: XTAL_GND, Crystal:Crystal_SMD_SeikoEpson_FA238-4Pin_3.2x2.5mm_HandSoldering
- added C6: 0.1u, Capacitor_SMD:C_0805_2012Metric, F.Cu at (513.9, -200.7)
- added R6: R, Capacitor_SMD:C_0805_2012Metric, F.Cu at (495.6, -183.0)
- added R7: R, Capacitor_SMD:C_0805_2012Metric, F.Cu at (502.6, -190.1)
- added U10: WS2812-2020, WS2812-2020:LED_WS2812-2020, F.Cu at (184.8, 4.06)
- added U100: WS2812-2020, WS2812-2020:LED_WS2812-2020, F.Cu at (510.3, -207.5)
- added U101: WS2812-2020, WS2812-2020:LED_WS2812-2020, F.Cu at (500.7, -196.9)
- added U102: WS2812-2020, WS2812-2020:LED_WS2812-2020, F.Cu at (482.3, -179.1)
- added U103: WS2812-2020, WS2812-2020:LED_WS2812-2020, F.Cu at (489.3, -186.2)
- added U104: WS2812-2020, WS2812-2020:LED_WS2812-2020, F.Cu at (505.2, -196.9)
- added U105: WS2812-2020, WS2812-2020:LED_WS2812-2020, F.Cu at (486.8, -182.7)
- added U106: WS2812-2020, WS2812-2020:LED_WS2812-2020, F.Cu at (493.8, -189.8)
- added U107: WS2812-2020, WS2812-2020:LED_WS2812-2020, F.Cu at (496.1, -196.9)
- added U108: WS2812-2020, WS2812-2020:LED_WS2812-2020, F.Cu at (509.7, -204.0)
- added U109: WS2812-2020, WS2812-2020:LED_WS2812-2020, F.Cu at (498.4, -186.2)
- added U11: WS2812-2020, WS2812-2020:LED_WS2812-2020, F.Cu at (214.0, 4.06)
- added U110: WS2812-2020, WS2812-2020:LED_WS2812-2020, F.Cu at (491.3, -179.1)
- added U111: WS2812-2020, WS2812-2020:LED_WS2812-2020, F.Cu at (509.7, -196.9)
- added U112: WS2812-2020, WS2812-2020:LED_WS2812-2020, F.Cu at (505.2, -193.3)
- added U113: WS2812-2020, WS2812-2020:LED_WS2812-2020, F.Cu at (514.2, -204.0)
- added U114: WS2812-2020, WS2812-2020:LED_WS2812-2020, F.Cu at (491.3, -182.7)
- added U115: WS2812-2020, WS2812-2020:LED_WS2812-2020, F.Cu at (498.4, -189.8)
- added U116: WS2812-2020, WS2812-2020:LED_WS2812-2020, F.Cu at (509.7, -200.4)
- added U117: WS2812-2020, WS2812-2020:LED_WS2812-2020, F.Cu at (486.8, -179.1)
- added U118: WS2812-2020, WS2812-2020:LED_WS2812-2020, F.Cu at (493.8, -186.2)
- added U119: AMS1117-3.3, Package_TO_SOT_SMD:SOT-223-3_TabPin2, F.Cu at (397.0, 0.00)
- added U12: WS2812-2020, WS2812-2020:LED_WS2812-2020, F.Cu at (233.6, 4.06)
- added U13: WS2812-2020, WS2812-2020:LED_WS2812-2020, F.Cu at (252.9, 4.06)
- added U14: WS2812-2020, WS2812-2020:LED_WS2812-2020, F.Cu at (272.4, 4.06)
- added U15: WS2812-2020, WS2812-2020:LED_WS2812-2020, F.Cu at (296.8, 4.06)
- added U16: WS2812-2020, WS2812-2020:LED_WS2812-2020, F.Cu at (316.2, 4.06)
- added U17: WS2812-2020, WS2812-2020:LED_WS2812-2020, F.Cu at (335.8, 4.06)
- added U18: WS2812-2020, WS2812-2020:LED_WS2812-2020, F.Cu at (-0.38, 32.6)
- added U19: WS2812-2020, WS2812-2020:LED_WS2812-2020, F.Cu at (19.2, 32.6)
- added U2: WS2812-2020, WS2812-2020:LED_WS2812-2020, F.Cu at (-0.38, 4.06)
- added U20: WS2812-2020, WS2812-2020:LED_WS2812-2020, F.Cu at (38.7, 32.6)
- added U21: WS2812-2020, WS2812-2020:LED_WS2812-2020, F.Cu at (58.2, 32.6)
- added U22: WS2812-2020, WS2812-2020:LED_WS2812-2020, F.Cu at (77.5, 32.6)
- added U23: WS2812-2020, WS2812-2020:LED_WS2812-2020, F.Cu at (96.9, 32.6)
- added U24: WS2812-2020, WS2812-2020:LED_WS2812-2020, F.Cu at (116.5, 32.6)
- added U25: WS2812-2020, WS2812-2020:LED_WS2812-2020, F.Cu at (136.0, 32.6)
- added U26: WS2812-2020, WS2812-2020:LED_WS2812-2020, F.Cu at (155.4, 32.6)
- added U27: WS2812-2020, WS2812-2020:LED_WS2812-2020, F.Cu at (174.9, 32.6)
- added U28: WS2812-2020, WS2812-2020:LED_WS2812-2020, F.Cu at (194.3, 32.6)
- added U29: WS2812-2020, WS2812-2020:LED_WS2812-2020, F.Cu at (213.9, 32.6)
- added U3: WS2812-2020, WS2812-2020:LED_WS2812-2020, F.Cu at (38.6, 4.06)
- added U30: WS2812-2020, WS2812-2020:LED_WS2812-2020, F.Cu at (233.3, 32.6)
- added U31: WS2812-2020, WS2812-2020:LED_WS2812-2020, F.Cu at (262.5, 32.6)
- added U32: WS2812-2020, WS2812-2020:LED_WS2812-2020, F.Cu at (4.45, 51.7)
- added U33: WS2812-2020, WS2812-2020:LED_WS2812-2020, F.Cu at (28.7, 51.7)
- added U34: WS2812-2020, WS2812-2020:LED_WS2812-2020, F.Cu at (48.3, 51.7)
- added U35: WS2812-2020, WS2812-2020:LED_WS2812-2020, F.Cu at (67.7, 51.7)
- added U36: WS2812-2020, WS2812-2020:LED_WS2812-2020, F.Cu at (87.2, 51.7)
- added U37: WS2812-2020, WS2812-2020:LED_WS2812-2020, F.Cu at (106.7, 51.7)
- added U38: WS2812-2020, WS2812-2020:LED_WS2812-2020, F.Cu at (126.2, 51.7)
- added U39: WS2812-2020, WS2812-2020:LED_WS2812-2020, F.Cu at (145.7, 51.7)
- added U4: WS2812-2020, WS2812-2020:LED_WS2812-2020, F.Cu at (58.0, 4.06)
- added U40: WS2812-2020, WS2812-2020:LED_WS2812-2020, F.Cu at (165.1, 51.7)
- added U41: WS2812-2020, WS2812-2020:LED_WS2812-2020, F.Cu at (184.7, 51.7)
- added U42: WS2812-2020, WS2812-2020:LED_WS2812-2020, F.Cu at (204.1, 51.7)
- added U43: WS2812-2020, WS2812-2020:LED_WS2812-2020, F.Cu at (223.6, 51.7)
- added U44: WS2812-2020, WS2812-2020:LED_WS2812-2020, F.Cu at (243.1, 51.7)
- added U45: WS2812-2020, WS2812-2020:LED_WS2812-2020, F.Cu at (267.5, 51.7)
- added U46: WS2812-2020, WS2812-2020:LED_WS2812-2020, F.Cu at (478.1, -196.9)
- added U47: WS2812-2020, WS2812-2020:LED_WS2812-2020, F.Cu at (487.7, -207.5)
- added U48: WS2812-2020, WS2812-2020:LED_WS2812-2020, F.Cu at (492.2, -211.1)
- added U49: WS2812-2020, WS2812-2020:LED_WS2812-2020, F.Cu at (495.2, -214.6)
- added U5: WS2812-2020, WS2812-2020:LED_WS2812-2020, F.Cu at (77.6, 4.06)
- added U50: WS2812-2020, WS2812-2020:LED_WS2812-2020, F.Cu at (482.6, -200.4)
- added U51: WS2812-2020, WS2812-2020:LED_WS2812-2020, F.Cu at (466.8, -183.3)
- added U52: WS2812-2020, WS2812-2020:LED_WS2812-2020, F.Cu at (473.6, -190.4)
- added U53: WS2812-2020, WS2812-2020:LED_WS2812-2020, F.Cu at (487.1, -204.0)
- added U54: WS2812-2020, WS2812-2020:LED_WS2812-2020, F.Cu at (471.3, -186.9)
- added U55: WS2812-2020, WS2812-2020:LED_WS2812-2020, F.Cu at (464.3, -179.8)
- added U56: WS2812-2020, WS2812-2020:LED_WS2812-2020, F.Cu at (478.1, -193.3)
- added U57: WS2812-2020, WS2812-2020:LED_WS2812-2020, F.Cu at (505.2, -200.4)
- added U58: WS2812-2020, WS2812-2020:LED_WS2812-2020, F.Cu at (500.7, -193.3)
- added U59: WS2812-2020, WS2812-2020:LED_WS2812-2020, F.Cu at (482.6, -196.9)
- added U6: WS2812-2020, WS2812-2020:LED_WS2812-2020, F.Cu at (97.2, 4.06)
- added U60: WS2812-2020, WS2812-2020:LED_WS2812-2020, F.Cu at (499.7, -214.6)
- added U61: WS2812-2020, WS2812-2020:LED_WS2812-2020, F.Cu at (496.7, -211.1)
- added U62: WS2812-2020, WS2812-2020:LED_WS2812-2020, F.Cu at (487.1, -200.4)
- added U63: WS2812-2020, WS2812-2020:LED_WS2812-2020, F.Cu at (471.3, -183.3)
- added U64: WS2812-2020, WS2812-2020:LED_WS2812-2020, F.Cu at (491.6, -204.0)
- added U65: WS2812-2020, WS2812-2020:LED_WS2812-2020, F.Cu at (475.8, -186.9)
- added U66: WS2812-2020, WS2812-2020:LED_WS2812-2020, F.Cu at (468.8, -179.8)
- added U67: WS2812-2020, WS2812-2020:LED_WS2812-2020, F.Cu at (482.6, -193.3)
- added U68: WS2812-2020, WS2812-2020:LED_WS2812-2020, F.Cu at (496.7, -207.5)
- added U69: WS2812-2020, WS2812-2020:LED_WS2812-2020, F.Cu at (487.1, -196.9)
- added U7: WS2812-2020, WS2812-2020:LED_WS2812-2020, F.Cu at (126.4, 4.06)
- added U70: WS2812-2020, WS2812-2020:LED_WS2812-2020, F.Cu at (501.3, -211.1)
- added U71: WS2812-2020, WS2812-2020:LED_WS2812-2020, F.Cu at (504.2, -214.6)
- added U72: WS2812-2020, WS2812-2020:LED_WS2812-2020, F.Cu at (491.6, -200.4)
- added U73: WS2812-2020, WS2812-2020:LED_WS2812-2020, F.Cu at (464.6, -194.0)
- added U74: WS2812-2020, WS2812-2020:LED_WS2812-2020, F.Cu at (492.2, -207.5)
- added U75: WS2812-2020, WS2812-2020:LED_WS2812-2020, F.Cu at (480.3, -189.8)
- added U76: WS2812-2020, WS2812-2020:LED_WS2812-2020, F.Cu at (473.3, -179.8)
- added U77: WS2812-2020, WS2812-2020:LED_WS2812-2020, F.Cu at (487.1, -193.3)
- added U78: WS2812-2020, WS2812-2020:LED_WS2812-2020, F.Cu at (501.3, -207.5)
- added U79: WS2812-2020, WS2812-2020:LED_WS2812-2020, F.Cu at (491.6, -196.9)
- added U8: WS2812-2020, WS2812-2020:LED_WS2812-2020, F.Cu at (145.7, 4.06)
- added U80: WS2812-2020, WS2812-2020:LED_WS2812-2020, F.Cu at (480.3, -186.2)
- added U81: WS2812-2020, WS2812-2020:LED_WS2812-2020, F.Cu at (508.7, -214.6)
- added U82: WS2812-2020, WS2812-2020:LED_WS2812-2020, F.Cu at (505.8, -211.1)
- added U83: WS2812-2020, WS2812-2020:LED_WS2812-2020, F.Cu at (496.1, -200.4)
- added U84: WS2812-2020, WS2812-2020:LED_WS2812-2020, F.Cu at (484.8, -189.8)
- added U85: WS2812-2020, WS2812-2020:LED_WS2812-2020, F.Cu at (500.7, -204.0)
- added U86: WS2812-2020, WS2812-2020:LED_WS2812-2020, F.Cu at (477.8, -179.8)
- added U87: WS2812-2020, WS2812-2020:LED_WS2812-2020, F.Cu at (491.6, -193.3)
- added U88: WS2812-2020, WS2812-2020:LED_WS2812-2020, F.Cu at (505.8, -207.5)
- added U89: WS2812-2020, WS2812-2020:LED_WS2812-2020, F.Cu at (475.8, -183.3)
- added U9: WS2812-2020, WS2812-2020:LED_WS2812-2020, F.Cu at (165.2, 4.06)
- added U90: WS2812-2020, WS2812-2020:LED_WS2812-2020, F.Cu at (482.6, -204.0)
- added U91: WS2812-2020, WS2812-2020:LED_WS2812-2020, F.Cu at (484.8, -186.2)
- added U92: WS2812-2020, WS2812-2020:LED_WS2812-2020, F.Cu at (496.1, -204.0)
- added U93: WS2812-2020, WS2812-2020:LED_WS2812-2020, F.Cu at (510.3, -211.1)
- added U94: WS2812-2020, WS2812-2020:LED_WS2812-2020, F.Cu at (513.2, -214.6)
- added U95: WS2812-2020, WS2812-2020:LED_WS2812-2020, F.Cu at (500.7, -200.4)
- added U96: WS2812-2020, WS2812-2020:LED_WS2812-2020, F.Cu at (489.3, -189.8)
- added U97: WS2812-2020, WS2812-2020:LED_WS2812-2020, F.Cu at (505.2, -204.0)
- added U98: WS2812-2020, WS2812-2020:LED_WS2812-2020, F.Cu at (482.3, -182.7)
- added U99: WS2812-2020, WS2812-2020:LED_WS2812-2020, F.Cu at (496.1, -193.3)
- R1: value 10K -> R; footprint Resistor_SMD:R_0805_2012Metric -> Capacitor_SMD:C_0805_2012Metric; moved to F.Cu
- SW1: value SW_PUSH -> SW_SPST; footprint Button_Switch_SMD:SW_SPST_TL3342 -> Button_Switch_THT:SW_Slide_1P2T_CK_OS102011MS2Q; moved to F.Cu
- SW2: value SW_SPST -> SW_Push; footprint Button_Switch_THT:SW_Slide_1P2T_CK_OS102011MS2Q -> Button_Switch_THT:Push_E-Switch_KS01Q01
- U1: value ATMEGA32U4 -> STM32F070RBTx; footprint Package_QFP:TQFP-44_10x10mm_P0.8mm -> Package_QFP:LQFP-64_10x10mm_P0.5mm; moved to F.Cu
- moved R1 228.8 mm to (509.4, -193.6), turned to 0 degrees
- moved SW1 37.6 mm to (354.1, -6.60)
- moved SW2 20.8 mm to (417.8, 7.11)
- moved R3 11.5 mm to (411.6, 7.74), turned to 0 degrees
- moved R2 8.28 mm to (411.6, 4.79), turned to 0 degrees
- moved U1 1.06 mm to (371.1, -2.54)
- renumbered C6 to C7
Connections:
- R1 pad 1: VCC -> +5V
- R1 pad 2: Net-(R1-Pad2) -> +5V
- SW1 pad 1: GND -> +5V
- SW1 pad 2: Net-(R1-Pad2) -> Net-(SW1-Pad2)
- SW2 pad 1: Net-(R6-Pad2) -> Net-(R6-Pad1)
- SW2 pad 2: GND -> +5V
- U1 pad 1: Net-(R6-Pad2) -> +5V
- U1 pad 10: /row1 -> Net-(U1-Pad10)
- U1 pad 11: /row2 -> Net-(U1-Pad11)
- U1 pad 12: /row3 -> +3V3
- U1 pad 13: Net-(R1-Pad2) -> +5V
- U1 pad 14: VCC -> /row0
- U1 pad 15: GND -> /row1
- U1 pad 16: Net-(C7-Pad1) -> /row2
- U1 pad 17: Net-(C3-Pad1) -> /row3
- U1 pad 18: /row4 -> +3V3
- U1 pad 19: /row5 -> +5V
- U1 pad 2: VCC -> Net-(U1-Pad2)
- U1 pad 20: /row6 -> /row4
- U1 pad 21: /row7 -> /row5
- U1 pad 22: /col0 -> /row6
- U1 pad 23: GND -> /row7
- U1 pad 24: VCC -> Net-(U1-Pad24)
- U1 pad 26: Net-(U1-Pad26) -> /col0
- U1 pad 29: /col3 -> /col10
- U1 pad 3: Net-(R4-Pad2) -> Net-(U1-Pad3)
- U1 pad 30: /col4 -> /col11
- U1 pad 31: /col5 -> +3V3
- U1 pad 32: /col6 -> +5V
- U1 pad 33: Net-(R7-Pad1) -> /col12
- U1 pad 34: VCC -> Net-(U1-Pad34)
- U1 pad 35: GND -> Net-(U1-Pad35)
- U1 pad 36: /col7 -> Net-(U1-Pad36)
- U1 pad 37: /col8 -> Net-(U1-Pad37)
- U1 pad 38: /col9 -> Net-(U1-Pad38)
- U1 pad 39: /col10 -> Net-(U1-Pad39)
- U1 pad 4: Net-(R5-Pad2) -> Net-(U1-Pad4)
- U1 pad 40: /col11 -> Net-(U1-Pad40)
- U1 pad 41: /col12 -> Net-(U1-Pad41)
- U1 pad 43: GND -> Net-(U1-Pad43)
- U1 pad 44: VCC -> Net-(R4-Pad2)
- U1 pad 5: GND -> Net-(U1-Pad5)
- U1 pad 7: VCC -> +5V
- U1 pad 8: /LEDDATA -> Net-(SW1-Pad2)
- U1 pad 9: /row0 -> /LEDDATA

Commit message: routed with all leds + gerbers
Parts:
- removed the R6 at (420.5, -7.50)
- removed the R6 at (495.6, -183.0)
- removed the R7 at (382.5, -7.00)
- removed the R7 at (502.6, -190.1)
- added R6: R, Capacitor_SMD:C_0805_2012Metric, F.Cu at (385.2, 4.79)
- added R7: R, Capacitor_SMD:C_0805_2012Metric, F.Cu at (382.1, -9.40)
- moved U71 597.3 mm to (2.03, 108.7)
- moved U108 596.5 mm to (-8.13, 92.1), turned to 270 degrees
- moved U107 564.1 mm to (-8.13, 56.0), turned to 270 degrees
- moved U72 558.6 mm to (26.3, 108.6)
- moved U59 551.1 mm to (11.8, 89.7)
- moved U60 548.4 mm to (43.4, 89.7)
- moved U109 547.9 mm to (38.6, 111.9)
- moved U46 541.8 mm to (6.99, 70.7)
- moved U106 540.9 mm to (-8.13, 11.8), turned to 270 degrees
- moved U47 532.6 mm to (33.7, 70.7)
- moved U61 527.9 mm to (62.9, 89.7)
- moved U48 521.7 mm to (53.2, 70.7)
- moved U73 512.7 mm to (50.7, 108.6)
- moved U49 509.9 mm to (72.6, 70.7)
- moved U62 498.0 mm to (82.3, 89.7)
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Connections:
- R1 pad 1: +5V -> +3V3
- R1 pad 2: +5V -> GND
- SW1 pad 1: +5V -> +3V3
- SW2 pad 2: +5V -> +3V3
- U1 pad 1: +5V -> GND
- U1 pad 13: +5V -> GND
- U1 pad 19: +5V -> GND
- U1 pad 32: +5V -> GND
- U1 pad 48: +5V -> GND
- U1 pad 64: +5V -> GND
- U1 pad 7: +5V -> +3V3
- U10 pad 2: +5V -> GND
- U100 pad 2: +5V -> GND
- U101 pad 2: +5V -> GND
- U102 pad 2: +5V -> GND
- U103 pad 2: +5V -> GND
- U104 pad 2: +5V -> GND
- U105 pad 2: +5V -> GND
- U106 pad 2: +5V -> GND
- U107 pad 2: +5V -> GND
- U108 pad 2: +5V -> GND
- U109 pad 2: +5V -> GND
- U11 pad 2: +5V -> GND
- U110 pad 2: +5V -> GND
- U111 pad 2: +5V -> GND
- U112 pad 2: +5V -> GND
- U113 pad 2: +5V -> GND
- U114 pad 2: +5V -> GND
- U115 pad 2: +5V -> GND
- U116 pad 2: +5V -> GND
- U117 pad 2: +5V -> GND
- U118 pad 2: +5V -> GND
- U119 pad 1: +5V -> GND
- U12 pad 2: +5V -> GND
- U13 pad 2: +5V -> GND
- U14 pad 2: +5V -> GND
- U15 pad 2: +5V -> GND
- U16 pad 2: +5V -> GND
- U17 pad 2: +5V -> GND
- U18 pad 2: +5V -> GND
- U19 pad 2: +5V -> GND
- U2 pad 2: +5V -> GND
- U20 pad 2: +5V -> GND
- U21 pad 2: +5V -> GND
- U22 pad 2: +5V -> GND
- U23 pad 2: +5V -> GND
- U24 pad 2: +5V -> GND
- U25 pad 2: +5V -> GND
- U26 pad 2: +5V -> GND
- U27 pad 2: +5V -> GND
- U28 pad 2: +5V -> GND
- U29 pad 2: +5V -> GND
- U3 pad 2: +5V -> GND
- U30 pad 2: +5V -> GND
- U31 pad 2: +5V -> GND
- U32 pad 2: +5V -> GND
- U33 pad 2: +5V -> GND
- U34 pad 2: +5V -> GND
- U35 pad 2: +5V -> GND
- U36 pad 2: +5V -> GND
- U37 pad 2: +5V -> GND
- U38 pad 2: +5V -> GND
- U39 pad 2: +5V -> GND
- U4 pad 2: +5V -> GND
- U40 pad 2: +5V -> GND
- U41 pad 2: +5V -> GND
- U42 pad 2: +5V -> GND
- U43 pad 2: +5V -> GND
- U44 pad 2: +5V -> GND
- U45 pad 2: +5V -> GND
- U46 pad 2: +5V -> GND
- U47 pad 2: +5V -> GND
- U48 pad 2: +5V -> GND
- U49 pad 2: +5V -> GND
- U5 pad 2: +5V -> GND
- U50 pad 2: +5V -> GND
- U51 pad 2: +5V -> GND
- U52 pad 2: +5V -> GND
- U53 pad 2: +5V -> GND
- U54 pad 2: +5V -> GND
- U55 pad 2: +5V -> GND
- U56 pad 2: +5V -> GND
- U57 pad 2: +5V -> GND
- U58 pad 2: +5V -> GND
- U59 pad 2: +5V -> GND
- U6 pad 2: +5V -> GND
- U60 pad 2: +5V -> GND
- U61 pad 2: +5V -> GND
- U62 pad 2: +5V -> GND
- U63 pad 2: +5V -> GND
- U64 pad 2: +5V -> GND
- U65 pad 2: +5V -> GND
- U66 pad 2: +5V -> GND
- U67 pad 2: +5V -> GND
- U68 pad 2: +5V -> GND
- U69 pad 2: +5V -> GND
- U7 pad 2: +5V -> GND
- U70 pad 2: +5V -> GND
- U71 pad 2: +5V -> GND
- U72 pad 2: +5V -> GND
- U73 pad 2: +5V -> GND
- U74 pad 2: +5V -> GND
- U75 pad 2: +5V -> GND
- U76 pad 2: +5V -> GND
- U77 pad 2: +5V -> GND
- U78 pad 2: +5V -> GND
- U79 pad 2: +5V -> GND
- U8 pad 2: +5V -> GND
- U80 pad 2: +5V -> GND
- U81 pad 2: +5V -> GND
- U82 pad 2: +5V -> GND
- U83 pad 2: +5V -> GND
- U84 pad 2: +5V -> GND
- U85 pad 2: +5V -> GND
- U86 pad 2: +5V -> GND
- U87 pad 2: +5V -> GND
- U88 pad 2: +5V -> GND
- U89 pad 2: +5V -> GND
- U9 pad 2: +5V -> GND
- U90 pad 2: +5V -> GND
- U91 pad 2: +5V -> GND
- U92 pad 2: +5V -> GND
- U93 pad 2: +5V -> GND
- U94 pad 2: +5V -> GND
- U95 pad 2: +5V -> GND
- U96 pad 2: +5V -> GND
- U97 pad 2: +5V -> GND
- U98 pad 2: +5V -> GND
- U99 pad 2: +5V -> GND
Routing:
- net GND: track 0.00 -> 2969.3 mm, vias 0 -> 76
- net VCC: track 0.00 -> 2230.9 mm, vias 0 -> 62
- net Net-(U104-Pad4): track 0.00 -> 1473.3 mm, vias 0 -> 30
- net /row1: track 0.00 -> 970.2 mm, vias 0 -> 16
- net /row6: track 0.00 -> 957.7 mm, vias 0 -> 17
- net /row0: track 0.00 -> 956.5 mm, vias 0 -> 14
- net /row5: track 0.00 -> 953.7 mm, vias 0 -> 16
- net /row7: track 0.00 -> 911.6 mm, vias 0 -> 15
- net /row4: track 0.00 -> 910.4 mm, vias 0 -> 19
- net /row2: track 0.00 -> 906.8 mm, vias 0 -> 17
- net /row3: track 0.00 -> 888.5 mm, vias 0 -> 21
- net Net-(U105-Pad1): track 0.00 -> 480.5 mm, vias 0 -> 2
- net /col8: track 0.00 -> 464.6 mm, vias 0 -> 3
- net /col5: track 0.00 -> 455.5 mm, vias 0 -> 7
- net /col7: track 0.00 -> 443.4 mm, vias 0 -> 6
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Other:
- board outline added: 444.5 x 132.1 mm
