File: keyboard/keyboard.sch (KiCad schematic (older format))
At the start: 18 parts, among them SW1 SW_PUSH, U1 ATMEGA32U4, X1 XTAL_GND

Commit message: add switches/leds
Parts:
- added D1, D10, D100, D101, D102, D103, D104, D11, D12, D13, D14, D15, D16, D17, D18, D19, D2, D20, D21, D22, D23, D24, D25, D26, D27, D28, D29, D3, D30, D31, D32, D33, D34, D35, D36, D37, D38, D39, D4, D40, D41, D42, D43, D44, D45, D46, D47, D48, D49, D5, D50, D51, D52, D53, D54, D55, D56, D57, D58, D59, D6, D60, D61, D62, D63, D64, D65, D66, D67, D68, D69, D7, D70, D71, D72, D73, D74, D75, D76, D77, D78, D79, D8, D80, D81, D82, D83, D84, D85, D86, D87, D88, D89, D9, D90, D91, D92, D93, D94, D95, D96, D97, D98, D99: D, keyboard1:D_SOD123_axial, symbol Device:D
- added D105, D106, D107, D108, D109, D110, D111, D112, D113, D114, D115, D116, D117, D118, D119, D120, D121, D122, D123, D124, D125, D126, D127, D128, D129, D130, D131, D132, D133, D134, D135, D136, D137, D138, D139, D140, D141, D142, D143, D144, D145, D146, D147, D148, D149, D150, D151, D152, D153, D154, D155, D156, D157, D158, D159, D160, D161, D162, D163, D164, D165, D166, D167, D168, D169, D170, D171, D172, D173, D174, D175, D176, D177, D178, D179, D180, D181, D182, D183, D184, D185, D186, D187, D188, D189, D190, D191, D192, D193, D194, D195, D196, D197, D198, D199, D200, D201, D202, D203, D204, D205, D206, D207, D208, D209, D210, D211, D212, D213, D214, D215, D216, D217, D218, D219, D220, D221, D222, D223, D224, D225, D226, D227, D228, D229, D230, D231, D232: SK6812MINI, LED_SMD:LED_SK6812MINI_PLCC4_3.5x3.5mm_P1.75mm, symbol LED:SK6812MINI
- added K1, K10, K100, K101, K102, K103, K104, K11, K12, K13, K14, K15, K16, K17, K18, K19, K2, K20, K21, K22, K23, K24, K25, K26, K27, K28, K29, K3, K30, K31, K32, K33, K34, K35, K36, K37, K38, K39, K4, K40, K41, K42, K43, K44, K45, K46, K47, K48, K49, K5, K50, K51, K52, K53, K54, K55, K56, K57, K58, K59, K6, K60, K61, K62, K63, K64, K65, K66, K67, K68, K69, K7, K70, K71, K72, K73, K74, K75, K76, K77, K78, K79, K8, K80, K81, K82, K83, K84, K85, K86, K87, K88, K89, K9, K90, K91, K92, K93, K94, K95, K96, K97, K98, K99: KEYSW, keyboard:Mx_Alps_100, symbol keyboard:KEYSW
- added R6: 10K, Resistor_SMD:R_0805_2012Metric, symbol keyboard:R
- added SW2: SW_SPST, Button_Switch_THT:SW_Slide_1P2T_CK_OS102011MS2Q, symbol Switch:SW_SPST
- C1: renamed from C3; footprint (none) -> Capacitor_SMD:C_0805_2012Metric
- C2: renamed from C4; footprint (none) -> Capacitor_SMD:C_0805_2012Metric
- C3: renamed from C1; footprint (none) -> Capacitor_SMD:C_0805_2012Metric
- C4: renamed from C5; footprint (none) -> Capacitor_SMD:C_0805_2012Metric
- C5: renamed from C6; footprint (none) -> Capacitor_SMD:C_0805_2012Metric
- C6: renamed from C7; footprint (none) -> Capacitor_SMD:C_0805_2012Metric
- C7: renamed from C2; footprint (none) -> Capacitor_SMD:C_0805_2012Metric
- C8: footprint (none) -> Capacitor_SMD:C_0805_2012Metric
- P1: renamed from P?; footprint (none) -> Connector_USB:USB_C_Receptacle_Amphenol_12401548E4-2A
- R1: footprint (none) -> Resistor_SMD:R_0805_2012Metric
- R2: renamed from R5; footprint (none) -> Resistor_SMD:R_0805_2012Metric
- R3: renamed from R6; footprint (none) -> Resistor_SMD:R_0805_2012Metric
- R4: renamed from R3; footprint (none) -> Resistor_SMD:R_0805_2012Metric
- R5: renamed from R4; footprint (none) -> Resistor_SMD:R_0805_2012Metric
- R7: renamed from R2; footprint (none) -> Resistor_SMD:R_0805_2012Metric
- SW1: footprint (none) -> Button_Switch_SMD:SW_SPST_TL3342
- U1: footprint (none) -> Package_QFP:TQFP-44_10x10mm_P0.8mm
- X1: footprint (none) -> Crystal:Crystal_SMD_SeikoEpson_FA238-4Pin_3.2x2.5mm_HandSoldering
Connections:
- net GND: now also D105.2 (VSS), D106.2 (VSS), D107.2 (VSS), D108.2 (VSS), D109.2 (VSS), D110.2 (VSS), D111.2 (VSS), D112.2 (VSS), D113.2 (VSS), D114.2 (VSS), D115.2 (VSS), D116.2 (VSS), D117.2 (VSS), D118.2 (VSS), D119.2 (VSS), D120.2 (VSS), D121.2 (VSS), D122.2 (VSS), D123.2 (VSS), D124.2 (VSS), D125.2 (VSS), D126.2 (VSS), D127.2 (VSS), D128.2 (VSS), D129.2 (VSS), D130.2 (VSS), D131.2 (VSS), D132.2 (VSS), D133.2 (VSS), D134.2 (VSS), D135.2 (VSS), D136.2 (VSS), D137.2 (VSS), D138.2 (VSS), D139.2 (VSS), D140.2 (VSS), D141.2 (VSS), D142.2 (VSS), D143.2 (VSS), D144.2 (VSS), D145.2 (VSS), D146.2 (VSS), D147.2 (VSS), D148.2 (VSS), D149.2 (VSS), D150.2 (VSS), D151.2 (VSS), D152.2 (VSS), D153.2 (VSS), D154.2 (VSS), D155.2 (VSS), D156.2 (VSS), D157.2 (VSS), D158.2 (VSS), D159.2 (VSS), D160.2 (VSS), D161.2 (VSS), D162.2 (VSS), D163.2 (VSS), D164.2 (VSS), D165.2 (VSS), D166.2 (VSS), D167.2 (VSS), D168.2 (VSS), D169.2 (VSS), D170.2 (VSS), D171.2 (VSS), D172.2 (VSS), D173.2 (VSS), D174.2 (VSS), D175.2 (VSS), D176.2 (VSS), D177.2 (VSS), D178.2 (VSS), D179.2 (VSS), D180.2 (VSS), D181.2 (VSS), D182.2 (VSS), D183.2 (VSS), D184.2 (VSS), D185.2 (VSS), D186.2 (VSS), D187.2 (VSS), D188.2 (VSS), D189.2 (VSS), D190.2 (VSS), D191.2 (VSS), D192.2 (VSS), D193.2 (VSS), D194.2 (VSS), D195.2 (VSS), D196.2 (VSS), D197.2 (VSS), D198.2 (VSS), D199.2 (VSS), D200.2 (VSS), D201.2 (VSS), D202.2 (VSS), D203.2 (VSS), D204.2 (VSS), D205.2 (VSS), D206.2 (VSS), D207.2 (VSS), D208.2 (VSS), D209.2 (VSS), D210.2 (VSS), D211.2 (VSS), D212.2 (VSS), D213.2 (VSS), D214.2 (VSS), D215.2 (VSS), D216.2 (VSS), D217.2 (VSS), D218.2 (VSS), D219.2 (VSS), D220.2 (VSS), D221.2 (VSS), D222.2 (VSS), D223.2 (VSS), D224.2 (VSS), D225.2 (VSS), D226.2 (VSS), D227.2 (VSS), D228.2 (VSS), D229.2 (VSS), D230.2 (VSS), D231.2 (VSS), D232.2 (VSS), SW2.2 (B)
- net VCC: now also U1.7 (VBus), D105.4 (VDD), D106.4 (VDD), D107.4 (VDD), D108.4 (VDD), D109.4 (VDD), D110.4 (VDD), D111.4 (VDD), D112.4 (VDD), D113.4 (VDD), D114.4 (VDD), D115.4 (VDD), D116.4 (VDD), D117.4 (VDD), D118.4 (VDD), D119.4 (VDD), D120.4 (VDD), D121.4 (VDD), D122.4 (VDD), D123.4 (VDD), D124.4 (VDD), D125.4 (VDD), D126.4 (VDD), D127.4 (VDD), D128.4 (VDD), D129.4 (VDD), D130.4 (VDD), D131.4 (VDD), D132.4 (VDD), D133.4 (VDD), D134.4 (VDD), D135.4 (VDD), D136.4 (VDD), D137.4 (VDD), D138.4 (VDD), D139.4 (VDD), D140.4 (VDD), D141.4 (VDD), D142.4 (VDD), D143.4 (VDD), D144.4 (VDD), D145.4 (VDD), D146.4 (VDD), D147.4 (VDD), D148.4 (VDD), D149.4 (VDD), D150.4 (VDD), D151.4 (VDD), D152.4 (VDD), D153.4 (VDD), D154.4 (VDD), D155.4 (VDD), D156.4 (VDD), D157.4 (VDD), D158.4 (VDD), D159.4 (VDD), D160.4 (VDD), D161.4 (VDD), D162.4 (VDD), D163.4 (VDD), D164.4 (VDD), D165.4 (VDD), D166.4 (VDD), D167.4 (VDD), D168.4 (VDD), D169.4 (VDD), D170.4 (VDD), D171.4 (VDD), D172.4 (VDD), D173.4 (VDD), D174.4 (VDD), D175.4 (VDD), D176.4 (VDD), D177.4 (VDD), D178.4 (VDD), D179.4 (VDD), D180.4 (VDD), D181.4 (VDD), D182.4 (VDD), D183.4 (VDD), D184.4 (VDD), D185.4 (VDD), D186.4 (VDD), D187.4 (VDD), D188.4 (VDD), D189.4 (VDD), D190.4 (VDD), D191.4 (VDD), D192.4 (VDD), D193.4 (VDD), D194.4 (VDD), D195.4 (VDD), D196.4 (VDD), D197.4 (VDD), D198.4 (VDD), D199.4 (VDD), D200.4 (VDD), D201.4 (VDD), D202.4 (VDD), D203.4 (VDD), D204.4 (VDD), D205.4 (VDD), D206.4 (VDD), D207.4 (VDD), D208.4 (VDD), D209.4 (VDD), D210.4 (VDD), D211.4 (VDD), D212.4 (VDD), D213.4 (VDD), D214.4 (VDD), D215.4 (VDD), D216.4 (VDD), D217.4 (VDD), D218.4 (VDD), D219.4 (VDD), D220.4 (VDD), D221.4 (VDD), D222.4 (VDD), D223.4 (VDD), D224.4 (VDD), D225.4 (VDD), D226.4 (VDD), D227.4 (VDD), D228.4 (VDD), D229.4 (VDD), D230.4 (VDD), D231.4 (VDD), D232.4 (VDD), R6.1
- net at U1.1 (PE6/AIN0): now also R6.2, SW2.1 (A)
- net row1: now reaches U1.10 (PB2/MOSI)
- net row1: now also D10.1 (K), D18.1 (K), D2.1 (K), D26.1 (K), D34.1 (K), D42.1 (K), D50.1 (K), D58.1 (K), D66.1 (K), D74.1 (K), D82.1 (K), D90.1 (K), D98.1 (K)
- net row2: now reaches U1.11 (PB3/MISO)
- net row2: now also D11.1 (K), D19.1 (K), D27.1 (K), D3.1 (K), D35.1 (K), D43.1 (K), D51.1 (K), D59.1 (K), D67.1 (K), D75.1 (K), D83.1 (K), D91.1 (K), D99.1 (K)
- net row3: now reaches U1.12 (PB7/~RTS)
- net row3: now also D100.1 (K), D12.1 (K), D20.1 (K), D28.1 (K), D36.1 (K), D4.1 (K), D44.1 (K), D52.1 (K), D60.1 (K), D68.1 (K), D76.1 (K), D84.1 (K), D92.1 (K)
- net row4: now reaches U1.18 (PD0/INT0)
- net row4: now also D101.1 (K), D13.1 (K), D21.1 (K), D29.1 (K), D37.1 (K), D45.1 (K), D5.1 (K), D53.1 (K), D61.1 (K), D69.1 (K), D77.1 (K), D85.1 (K), D93.1 (K)
- net row5: now reaches U1.19 (PD1/INT1)
- net row5: now also D102.1 (K), D14.1 (K), D22.1 (K), D30.1 (K), D38.1 (K), D46.1 (K), D54.1 (K), D6.1 (K), D62.1 (K), D70.1 (K), D78.1 (K), D86.1 (K), D94.1 (K)
- net row6: now reaches U1.20 (PD2/RXD1)
- net row6: now also D103.1 (K), D15.1 (K), D23.1 (K), D31.1 (K), D39.1 (K), D47.1 (K), D55.1 (K), D63.1 (K), D7.1 (K), D71.1 (K), D79.1 (K), D87.1 (K), D95.1 (K)
- net row7: now reaches U1.21 (PD3/TXD1)
- net row7: now also D104.1 (K), D16.1 (K), D24.1 (K), D32.1 (K), D40.1 (K), D48.1 (K), D56.1 (K), D64.1 (K), D72.1 (K), D8.1 (K), D80.1 (K), D88.1 (K), D96.1 (K)
- net col0: now reaches U1.22 (PD5/XCK1)
- net col0: now also K1.1, K2.1, K3.1, K4.1, K5.1, K6.1, K7.1, K8.1
- net col1: now reaches U1.27 (T0/PD7)
- net col1: now also K10.1, K11.1, K12.1, K13.1, K14.1, K15.1, K16.1, K9.1
- net col2: now reaches U1.28 (PB4)
- net col2: now also K17.1, K18.1, K19.1, K20.1, K21.1, K22.1, K23.1, K24.1
- net col3: now reaches U1.29 (PB5)
- net col3: now also K25.1, K26.1, K27.1, K28.1, K29.1, K30.1, K31.1, K32.1
- net col4: now reaches U1.30 (PB6)
- net col4: now also K33.1, K34.1, K35.1, K36.1, K37.1, K38.1, K39.1, K40.1
- net col5: now reaches U1.31 (PC6)
- net col5: now also K41.1, K42.1, K43.1, K44.1, K45.1, K46.1, K47.1, K48.1
- net col6: now reaches U1.32 (PC7)
- net col6: now also K49.1, K50.1, K51.1, K52.1, K53.1, K54.1, K55.1, K56.1
- net col7: now reaches U1.36 (PF7)
- net col7: now also K57.1, K58.1, K59.1, K60.1, K61.1, K62.1, K63.1, K64.1
- net col8: now reaches U1.37 (PF6)
- net col8: now also K65.1, K66.1, K67.1, K68.1, K69.1, K70.1, K71.1, K72.1
- net col9: now reaches U1.38 (PF5)
- net col9: now also K73.1, K74.1, K75.1, K76.1, K77.1, K78.1, K79.1, K80.1
- net col10: now reaches U1.39 (PF4)
- net col10: now also K81.1, K82.1, K83.1, K84.1, K85.1, K86.1, K87.1, K88.1
- net col11: now reaches U1.40 (PF1)
- net col11: now also K89.1, K90.1, K91.1, K92.1, K93.1, K94.1, K95.1, K96.1
- net col12: now reaches U1.41 (PF0)
- net col12: now also K100.1, K101.1, K102.1, K103.1, K104.1, K97.1, K98.1, K99.1
- net LEDDATA: now reaches U1.8 (PB0/SS)
- net LEDDATA: now also D105.3 (DIN)
- net row0: now reaches U1.9 (PB1/SCK)
- net row0: now also D1.1 (K), D17.1 (K), D25.1 (K), D33.1 (K), D41.1 (K), D49.1 (K), D57.1 (K), D65.1 (K), D73.1 (K), D81.1 (K), D89.1 (K), D9.1 (K), D97.1 (K)
- new net: D1.2 (A), K1.2
- new net: D9.2 (A), K9.2
- new net: D17.2 (A), K17.2
- new net: D25.2 (A), K25.2
- new net: D33.2 (A), K33.2
- new net: D41.2 (A), K41.2
- new net: D49.2 (A), K49.2
- new net: D57.2 (A), K57.2
- new net: D65.2 (A), K65.2
- new net: D73.2 (A), K73.2
- new net: D81.2 (A), K81.2
- new net: D89.2 (A), K89.2
- new net: D97.2 (A), K97.2
- new net: D2.2 (A), K2.2
- new net: D10.2 (A), K10.2
- new net: D18.2 (A), K18.2
- new net: D26.2 (A), K26.2
- new net: D34.2 (A), K34.2
- new net: D42.2 (A), K42.2
- new net: D50.2 (A), K50.2
- new net: D58.2 (A), K58.2
- new net: D66.2 (A), K66.2
- new net: D74.2 (A), K74.2
- new net: D82.2 (A), K82.2
- new net: D90.2 (A), K90.2
- new net: D98.2 (A), K98.2
- new net: D3.2 (A), K3.2
- new net: D11.2 (A), K11.2
- new net: D19.2 (A), K19.2
- new net: D27.2 (A), K27.2
- new net: D35.2 (A), K35.2
- new net: D43.2 (A), K43.2
- new net: D51.2 (A), K51.2
- new net: D59.2 (A), K59.2
- new net: D67.2 (A), K67.2
- new net: D75.2 (A), K75.2
- new net: D83.2 (A), K83.2
- new net: D91.2 (A), K91.2
- new net: D99.2 (A), K99.2
- new net: D4.2 (A), K4.2
- new net: D12.2 (A), K12.2
- new net: D20.2 (A), K20.2
- new net: D28.2 (A), K28.2
- new net: D36.2 (A), K36.2
- new net: D44.2 (A), K44.2
- new net: D52.2 (A), K52.2
- new net: D60.2 (A), K60.2
- new net: D68.2 (A), K68.2
- new net: D76.2 (A), K76.2
- new net: D84.2 (A), K84.2
- new net: D92.2 (A), K92.2
- new net: D100.2 (A), K100.2
- new net: D5.2 (A), K5.2
- new net: D13.2 (A), K13.2
- new net: D21.2 (A), K21.2
- new net: D29.2 (A), K29.2
- new net: D37.2 (A), K37.2
- new net: D45.2 (A), K45.2
- new net: D53.2 (A), K53.2
- new net: D61.2 (A), K61.2
- new net: D69.2 (A), K69.2
- new net: D77.2 (A), K77.2
- new net: D85.2 (A), K85.2
- new net: D93.2 (A), K93.2
- new net: D101.2 (A), K101.2
- new net: D6.2 (A), K6.2
- new net: D14.2 (A), K14.2
- new net: D22.2 (A), K22.2
- new net: D30.2 (A), K30.2
- new net: D38.2 (A), K38.2
- new net: D46.2 (A), K46.2
- new net: D54.2 (A), K54.2
- new net: D62.2 (A), K62.2
- new net: D70.2 (A), K70.2
- new net: D78.2 (A), K78.2
- new net: D86.2 (A), K86.2
- new net: D94.2 (A), K94.2
- new net: D102.2 (A), K102.2
- new net: D7.2 (A), K7.2
- new net: D15.2 (A), K15.2
- new net: D23.2 (A), K23.2
- new net: D31.2 (A), K31.2
- new net: D39.2 (A), K39.2
- new net: D47.2 (A), K47.2
- new net: D55.2 (A), K55.2
- new net: D63.2 (A), K63.2
- new net: D71.2 (A), K71.2
- new net: D79.2 (A), K79.2
- new net: D87.2 (A), K87.2
- new net: D95.2 (A), K95.2
- new net: D103.2 (A), K103.2
- new net: D8.2 (A), K8.2
- new net: D16.2 (A), K16.2
- new net: D24.2 (A), K24.2
- new net: D32.2 (A), K32.2
- new net: D40.2 (A), K40.2
- new net: D48.2 (A), K48.2
- new net: D56.2 (A), K56.2
- new net: D64.2 (A), K64.2
- new net: D72.2 (A), K72.2
- new net: D80.2 (A), K80.2
- new net: D88.2 (A), K88.2
- new net: D96.2 (A), K96.2
- new net: D104.2 (A), K104.2
- new net: D106.1 (DOUT), D114.3 (DIN)
- new net: D106.3 (DIN), D225.1 (DOUT)
- new net: D114.1 (DOUT), D122.3 (DIN)
- new net: D122.1 (DOUT), D130.3 (DIN)
- new net: D130.1 (DOUT), D138.3 (DIN)
- new net: D138.1 (DOUT), D146.3 (DIN)
- new net: D146.1 (DOUT), D154.3 (DIN)
- new net: D154.1 (DOUT), D162.3 (DIN)
- new net: D162.1 (DOUT), D170.3 (DIN)
- new net: D170.1 (DOUT), D178.3 (DIN)
- new net: D178.1 (DOUT), D186.3 (DIN)
- new net: D186.1 (DOUT), D194.3 (DIN)
- new net: D194.1 (DOUT), D202.3 (DIN)
- new net: D202.1 (DOUT), D210.3 (DIN)
- new net: D210.1 (DOUT), D218.3 (DIN)
- new net: D218.1 (DOUT), D226.3 (DIN)
- new net: D107.3 (DIN), D226.1 (DOUT)
- new net: D107.1 (DOUT), D115.3 (DIN)
- new net: D115.1 (DOUT), D123.3 (DIN)
- new net: D123.1 (DOUT), D131.3 (DIN)
- new net: D131.1 (DOUT), D139.3 (DIN)
- new net: D139.1 (DOUT), D147.3 (DIN)
- new net: D147.1 (DOUT), D155.3 (DIN)
- new net: D155.1 (DOUT), D163.3 (DIN)
- new net: D163.1 (DOUT), D171.3 (DIN)
- new net: D171.1 (DOUT), D179.3 (DIN)
- new net: D179.1 (DOUT), D187.3 (DIN)
- new net: D187.1 (DOUT), D195.3 (DIN)
- new net: D195.1 (DOUT), D203.3 (DIN)
- new net: D203.1 (DOUT), D211.3 (DIN)
- new net: D211.1 (DOUT), D219.3 (DIN)
- new net: D219.1 (DOUT), D227.3 (DIN)
- new net: D108.3 (DIN), D227.1 (DOUT)
- new net: D108.1 (DOUT), D116.3 (DIN)
- new net: D116.1 (DOUT), D124.3 (DIN)
- new net: D124.1 (DOUT), D132.3 (DIN)
- new net: D132.1 (DOUT), D140.3 (DIN)
- new net: D140.1 (DOUT), D148.3 (DIN)
- new net: D148.1 (DOUT), D156.3 (DIN)
- new net: D156.1 (DOUT), D164.3 (DIN)
- new net: D164.1 (DOUT), D172.3 (DIN)
- new net: D172.1 (DOUT), D180.3 (DIN)
- new net: D180.1 (DOUT), D188.3 (DIN)
- new net: D188.1 (DOUT), D196.3 (DIN)
- new net: D196.1 (DOUT), D204.3 (DIN)
- new net: D204.1 (DOUT), D212.3 (DIN)
- new net: D212.1 (DOUT), D220.3 (DIN)
- new net: D220.1 (DOUT), D228.3 (DIN)
- new net: D109.3 (DIN), D228.1 (DOUT)
- new net: D109.1 (DOUT), D117.3 (DIN)
- new net: D117.1 (DOUT), D125.3 (DIN)
- new net: D125.1 (DOUT), D133.3 (DIN)
- new net: D133.1 (DOUT), D141.3 (DIN)
- new net: D141.1 (DOUT), D149.3 (DIN)
- new net: D149.1 (DOUT), D157.3 (DIN)
- new net: D157.1 (DOUT), D165.3 (DIN)
- new net: D165.1 (DOUT), D173.3 (DIN)
- new net: D173.1 (DOUT), D181.3 (DIN)
- new net: D181.1 (DOUT), D189.3 (DIN)
- new net: D189.1 (DOUT), D197.3 (DIN)
- new net: D197.1 (DOUT), D205.3 (DIN)
- new net: D205.1 (DOUT), D213.3 (DIN)
- new net: D213.1 (DOUT), D221.3 (DIN)
- new net: D221.1 (DOUT), D229.3 (DIN)
- new net: D110.3 (DIN), D229.1 (DOUT)
- new net: D110.1 (DOUT), D118.3 (DIN)
- new net: D118.1 (DOUT), D126.3 (DIN)
- new net: D126.1 (DOUT), D134.3 (DIN)
- new net: D134.1 (DOUT), D142.3 (DIN)
- new net: D142.1 (DOUT), D150.3 (DIN)
- new net: D150.1 (DOUT), D158.3 (DIN)
- new net: D158.1 (DOUT), D166.3 (DIN)
- new net: D166.1 (DOUT), D174.3 (DIN)
- new net: D174.1 (DOUT), D182.3 (DIN)
- new net: D182.1 (DOUT), D190.3 (DIN)
- new net: D190.1 (DOUT), D198.3 (DIN)
- new net: D198.1 (DOUT), D206.3 (DIN)
- new net: D206.1 (DOUT), D214.3 (DIN)
- new net: D214.1 (DOUT), D222.3 (DIN)
- new net: D222.1 (DOUT), D230.3 (DIN)
- new net: D111.3 (DIN), D230.1 (DOUT)
- new net: D111.1 (DOUT), D119.3 (DIN)
- new net: D119.1 (DOUT), D127.3 (DIN)
- new net: D127.1 (DOUT), D135.3 (DIN)
- new net: D135.1 (DOUT), D143.3 (DIN)
- new net: D143.1 (DOUT), D151.3 (DIN)
- new net: D151.1 (DOUT), D159.3 (DIN)
- new net: D159.1 (DOUT), D167.3 (DIN)
- new net: D167.1 (DOUT), D175.3 (DIN)
- new net: D175.1 (DOUT), D183.3 (DIN)
- new net: D183.1 (DOUT), D191.3 (DIN)
- new net: D191.1 (DOUT), D199.3 (DIN)
- new net: D199.1 (DOUT), D207.3 (DIN)
- new net: D207.1 (DOUT), D215.3 (DIN)
- new net: D215.1 (DOUT), D223.3 (DIN)
- new net: D223.1 (DOUT), D231.3 (DIN)
- new net: D112.3 (DIN), D231.1 (DOUT)
- new net: D112.1 (DOUT), D120.3 (DIN)
- new net: D120.1 (DOUT), D128.3 (DIN)
- new net: D128.1 (DOUT), D136.3 (DIN)
- new net: D136.1 (DOUT), D144.3 (DIN)
- new net: D144.1 (DOUT), D152.3 (DIN)
- new net: D152.1 (DOUT), D160.3 (DIN)
- new net: D160.1 (DOUT), D168.3 (DIN)
- new net: D168.1 (DOUT), D176.3 (DIN)
- new net: D176.1 (DOUT), D184.3 (DIN)
- new net: D184.1 (DOUT), D192.3 (DIN)
- new net: D192.1 (DOUT), D200.3 (DIN)
- new net: D200.1 (DOUT), D208.3 (DIN)
- new net: D208.1 (DOUT), D216.3 (DIN)
- new net: D216.1 (DOUT), D224.3 (DIN)
- new net: D224.1 (DOUT), D232.3 (DIN)
- new net: D105.1 (DOUT), D113.3 (DIN)
- new net: D113.1 (DOUT), D121.3 (DIN)
- new net: D121.1 (DOUT), D129.3 (DIN)
- new net: D129.1 (DOUT), D137.3 (DIN)
- new net: D137.1 (DOUT), D145.3 (DIN)
- new net: D145.1 (DOUT), D153.3 (DIN)
- new net: D153.1 (DOUT), D161.3 (DIN)
- new net: D161.1 (DOUT), D169.3 (DIN)
- new net: D169.1 (DOUT), D177.3 (DIN)
- new net: D177.1 (DOUT), D185.3 (DIN)
- new net: D185.1 (DOUT), D193.3 (DIN)
- new net: D193.1 (DOUT), D201.3 (DIN)
- new net: D201.1 (DOUT), D209.3 (DIN)
- new net: D209.1 (DOUT), D217.3 (DIN)
- new net: D217.1 (DOUT), D225.3 (DIN)
- no-connect marks 0 -> 4
Other:
- note added: "23 pins free for matrix input - 132 keys MAX"
- moved on the sheet: C1, C2, C3, C4, C5, C6, C7, C8, P1, R1, R2, R3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

Commit message: arrange switches/diodes/other
Connections:
- net at C3.1, X1.1: now also U1.17 (XTAL2); no longer U1.16 (XTAL1)
- net at C7.1, X1.2: now also U1.16 (XTAL1); no longer U1.17 (XTAL2)
Changed lines of the file:
@@
 $EndComp
 $Comp
-L keyboard:XTAL_GND X1
-U 1 1 5D720272
-P 3100 5450
-F 0 "X1" H 3100 5742 60  0000 C CNN
-F 1 "XTAL_GND" H 3100 5636 60  0000 C CNN
-F 2 "Crystal:Crystal_SMD_SeikoEpson_FA238-4Pin_3.2x2.5mm_HandSoldering" H 3100 5450 60  0001 C CNN
-F 3 "" H 3100 5450 60  0000 C CNN
-	1    3100 5450
-	1    0    0    -1
-$EndComp
-$Comp
 L Device:C_Small C3
 U 1 1 5D720D23
@@
 $EndComp
 Wire Wire Line
-	3100 5900 3100 5650
-Wire Wire Line
 	3600 5800 3600 5900
 Wire Wire Line
@@
 	2600 5450 2600 5550
 Wire Wire Line
-	4150 5300 3600 5300
-Wire Wire Line
-	3600 5300 3600 5450
-Wire Wire Line
 	3600 5450 3400 5450
-Connection ~ 3600 5450
 Wire Wire Line
 	3600 5450 3600 5600
-Wire Wire Line
-	4150 5200 2600 5200
-Wire Wire Line
-	2600 5200 2600 5450
-Connection ~ 2600 5450
 $Comp
 L power:VCC #PWR01
@@
 Wire Wire Line
 	11350 13450 12050 13450
+Wire Wire Line
+	3100 5650 3100 5900
+$Comp
+L keyboard:XTAL_GND X1
+U 1 1 5D720272
+P 3100 5450
+F 0 "X1" H 3100 5742 60  0000 C CNN
+F 1 "XTAL_GND" H 3100 5636 60  0000 C CNN
+F 2 "Crystal:Crystal_SMD_SeikoEpson_FA238-4Pin_3.2x2.5mm_HandSoldering" H 3100 5450 60  0001 C CNN
+F 3 "" H 3100 5450 60  0000 C CNN
+	1    3100 5450
+	1    0    0    -1
+$EndComp
+Wire Wire Line
+	3600 5450 3600 5200
+Wire Wire Line
+	3600 5200 4150 5200
+Connection ~ 3600 5450
+Wire Wire Line
+	4150 5300 2600 5300
+Wire Wire Line
+	2600 5300 2600 5450
+Connection ~ 2600 5450
 $EndSCHEMATC

Commit message: add datasheets
Parts:
- removed C3, C7: 22p, Capacitor_SMD:C_0805_2012Metric, symbol Device:C_Small
- removed C8: 1u, Capacitor_SMD:C_0805_2012Metric, symbol Device:C_Small
- removed D105, D106, D107, D108, D109, D110, D111, D112, D113, D114, D115, D116, D117, D118, D119, D120, D121, D122, D123, D124, D125, D126, D127, D128, D129, D130, D131, D132, D133, D134, D135, D136, D137, D138, D139, D140, D141, D142, D143, D144, D145, D146, D147, D148, D149, D150, D151, D152, D153, D154, D155, D156, D157, D158, D159, D160, D161, D162, D163, D164, D165, D166, D167, D168, D169, D170, D171, D172, D173, D174, D175, D176, D177, D178, D179, D180, D181, D182, D183, D184, D185, D186, D187, D188, D189, D190, D191, D192, D193, D194, D195, D196, D197, D198, D199, D200, D201, D202, D203, D204, D205, D206, D207, D208, D209, D210, D211, D212, D213, D214, D215, D216, D217, D218, D219, D220, D221, D222, D223, D224, D225, D226, D227, D228, D229, D230, D231, D232: SK6812MINI, LED_SMD:LED_SK6812MINI_PLCC4_3.5x3.5mm_P1.75mm, symbol LED:SK6812MINI
- removed R1, R6, R7: 10K, Resistor_SMD:R_0805_2012Metric, symbol keyboard:R
- removed SW1: SW_PUSH, Button_Switch_SMD:SW_SPST_TL3342, symbol keyboard:SW_PUSH
- removed SW2: SW_SPST, Button_Switch_THT:SW_Slide_1P2T_CK_OS102011MS2Q, symbol Switch:SW_SPST
- removed U1: ATMEGA32U4, Package_QFP:TQFP-44_10x10mm_P0.8mm, symbol keyboard:ATMEGA32U4
- removed X1: XTAL_GND, Crystal:Crystal_SMD_SeikoEpson_FA238-4Pin_3.2x2.5mm_HandSoldering, symbol keyboard:XTAL_GND
- added C6: 0.1u, symbol Device:C_Small
- added R?: R, symbol Device:R
- added SW?: SW_SPST, symbol Switch:SW_SPST
- added U1: STM32F070RBTx, Package_QFP:LQFP-64_10x10mm_P0.5mm, symbol MCU_ST_STM32F0:STM32F070RBTx
- added U2, U3, U4: IS31FL3733-TQ, Package_QFP:TQFP-48-1EP_7x7mm_P0.5mm_EP5x5mm, symbol Driver_LED:IS31FL3733-TQ
- renumbered C6 to C7
Connections:
- net GND: now also C6.2
- net VCC: now also C6.1
- net col0: now also U1.26 (PB0)
- net col1: now also U1.27 (PB1)
- net col10: now also U1.29 (PB10)
- net col11: now also U1.30 (PB11)
- net col12: now also U1.33 (PB12)
- net col2: now also U1.28 (PB2)
- net col3: now also U1.55 (PB3)
- net col4: now also U1.56 (PB4)
- net col5: now also U1.57 (PB5)
- net col6: now also U1.58 (PB6)
- net col7: now also U1.59 (PB7)
- net col8: now also U1.61 (PB8)
- net col9: now also U1.62 (PB9)
- net row0: now also U1.14 (PA0)
- net row1: now also U1.15 (PA1)
- net row2: now also U1.16 (PA2)
- net row3: now also U1.17 (PA3)
- net row4: now also U1.20 (PA4)
- net row5: now also U1.21 (PA5)
- net row6: now also U1.22 (PA6)
- net row7: now also U1.23 (PA7)
- new net: SW?.2 (B), U1.8 (PC0)
- new net: U2.12 (PGND), U2.5 (PGND)
- new net: U2.48 (GND), U2.49 (GND)
- new net: U3.12 (PGND), U3.5 (PGND)
- new net: U3.48 (GND), U3.49 (GND)
- new net: U4.12 (PGND), U4.5 (PGND)
- new net: U4.48 (GND), U4.49 (GND)
- new net +5V: R?.1, R?.2, SW?.1 (A)
- new net I2C1_SCL: U1.6 (PF1)
- new net I2C1_SDA: U1.5 (PF0)
- no-connect marks 4 -> 0
Other:
- moved on the sheet: C1, C2, C4, C5, C7

Commit message: finally figure out leds & remove led drivers
Parts:
- removed U2, U3, U4: IS31FL3733-TQ, Package_QFP:TQFP-48-1EP_7x7mm_P0.5mm_EP5x5mm, symbol Driver_LED:IS31FL3733-TQ
- added R6, R7: R, Capacitor_SMD:C_0805_2012Metric, symbol Device:R
- added SW2: SW_Push, Button_Switch_THT:Push_E-Switch_KS01Q01, symbol Switch:SW_Push
- added U10, U100, U101, U102, U103, U104, U105, U106, U107, U108, U109, U11, U110, U111, U112, U113, U114, U115, U116, U117, U118, U12, U13, U14, U15, U16, U17, U18, U19, U2, U20, U21, U22, U23, U24, U25, U26, U27, U28, U29, U3, U30, U31, U32, U33, U34, U35, U36, U37, U38, U39, U4, U40, U41, U42, U43, U44, U45, U46, U47, U48, U49, U5, U50, U51, U52, U53, U54, U55, U56, U57, U58, U59, U6, U60, U61, U62, U63, U64, U65, U66, U67, U68, U69, U7, U70, U71, U72, U73, U74, U75, U76, U77, U78, U79, U8, U80, U81, U82, U83, U84, U85, U86, U87, U88, U89, U9, U90, U91, U92, U93, U94, U95, U96, U97, U98, U99: WS2812-2020, WS2812-2020:LED_WS2812-2020, symbol WS2812-2020:WS2812-2020
- added U119: AMS1117-3.3, Package_TO_SOT_SMD:SOT-223-3_TabPin2, symbol Regulator_Linear:AMS1117-3.3
- C6: footprint (none) -> Capacitor_SMD:C_0805_2012Metric
- R1: renamed from R?; footprint (none) -> Capacitor_SMD:C_0805_2012Metric
- SW1: renamed from SW?; footprint (none) -> Button_Switch_THT:SW_Slide_1P2T_CK_OS102011MS2Q
Connections:
- net GND: now also R1.2, U1.1 (VDD), U1.13 (VDDA), U1.19 (VDD), U1.32 (VDD), U1.48 (VDD), U1.64 (VDD), R6.2, R7.2, U10.2 (GND), U100.2 (GND), U101.2 (GND), U102.2 (GND), U103.2 (GND), U104.2 (GND), U105.2 (GND), U106.2 (GND), U107.2 (GND), U108.2 (GND), U109.2 (GND), U11.2 (GND), U110.2 (GND), U111.2 (GND), U112.2 (GND), U113.2 (GND), U114.2 (GND), U115.2 (GND), U116.2 (GND), U117.2 (GND), U118.2 (GND), U119.1 (GND), U12.2 (GND), U13.2 (GND), U14.2 (GND), U15.2 (GND), U16.2 (GND), U17.2 (GND), U18.2 (GND), U19.2 (GND), U2.2 (GND), U20.2 (GND), U21.2 (GND), U22.2 (GND), U23.2 (GND), U24.2 (GND), U25.2 (GND), U26.2 (GND), U27.2 (GND), U28.2 (GND), U29.2 (GND), U3.2 (GND), U30.2 (GND), U31.2 (GND), U32.2 (GND), U33.2 (GND), U34.2 (GND), U35.2 (GND), U36.2 (GND), U37.2 (GND), U38.2 (GND), U39.2 (GND), U4.2 (GND), U40.2 (GND), U41.2 (GND), U42.2 (GND), U43.2 (GND), U44.2 (GND), U45.2 (GND), U46.2 (GND), U47.2 (GND), U48.2 (GND), U49.2 (GND), U5.2 (GND), U50.2 (GND), U51.2 (GND), U52.2 (GND), U53.2 (GND), U54.2 (GND), U55.2 (GND), U56.2 (GND), U57.2 (GND), U58.2 (GND), U59.2 (GND), U6.2 (GND), U60.2 (GND), U61.2 (GND), U62.2 (GND), U63.2 (GND), U64.2 (GND), U65.2 (GND), U66.2 (GND), U67.2 (GND), U68.2 (GND), U69.2 (GND), U7.2 (GND), U70.2 (GND), U71.2 (GND), U72.2 (GND), U73.2 (GND), U74.2 (GND), U75.2 (GND), U76.2 (GND), U77.2 (GND), U78.2 (GND), U79.2 (GND), U8.2 (GND), U80.2 (GND), U81.2 (GND), U82.2 (GND), U83.2 (GND), U84.2 (GND), U85.2 (GND), U86.2 (GND), U87.2 (GND), U88.2 (GND), U89.2 (GND), U9.2 (GND), U90.2 (GND), U91.2 (GND), U92.2 (GND), U93.2 (GND), U94.2 (GND), U95.2 (GND), U96.2 (GND), U97.2 (GND), U98.2 (GND), U99.2 (GND)
- net VCC: now also U10.4 (VDD), U100.4 (VDD), U101.4 (VDD), U102.4 (VDD), U103.4 (VDD), U11.4 (VDD), U119.3 (VI), U12.4 (VDD), U13.4 (VDD), U14.4 (VDD), U15.4 (VDD), U18.4 (VDD), U19.4 (VDD), U2.4 (VDD), U20.4 (VDD), U21.4 (VDD), U22.4 (VDD), U23.4 (VDD), U26.4 (VDD), U27.4 (VDD), U28.4 (VDD), U29.4 (VDD), U3.4 (VDD), U30.4 (VDD), U31.4 (VDD), U34.4 (VDD), U35.4 (VDD), U36.4 (VDD), U37.4 (VDD), U38.4 (VDD), U39.4 (VDD), U4.4 (VDD), U42.4 (VDD), U43.4 (VDD), U44.4 (VDD), U45.4 (VDD), U46.4 (VDD), U47.4 (VDD), U5.4 (VDD), U50.4 (VDD), U51.4 (VDD), U52.4 (VDD), U53.4 (VDD), U54.4 (VDD), U55.4 (VDD), U58.4 (VDD), U59.4 (VDD), U6.4 (VDD), U60.4 (VDD), U61.4 (VDD), U62.4 (VDD), U63.4 (VDD), U66.4 (VDD), U67.4 (VDD), U68.4 (VDD), U69.4 (VDD), U7.4 (VDD), U70.4 (VDD), U71.4 (VDD), U74.4 (VDD), U75.4 (VDD), U76.4 (VDD), U77.4 (VDD), U78.4 (VDD), U79.4 (VDD), U82.4 (VDD), U83.4 (VDD), U84.4 (VDD), U85.4 (VDD), U86.4 (VDD), U87.4 (VDD), U90.4 (VDD), U91.4 (VDD), U92.4 (VDD), U93.4 (VDD), U94.4 (VDD), U95.4 (VDD), U98.4 (VDD), U99.4 (VDD)
- net at R4.2: now also U1.44 (PA11)
- net at R5.2: now also U1.45 (PA12)
- net +3V3: now reaches U1.12 (VSSA)
- net +3V3: now also R1.1, SW1.1 (A), U1.18 (VSS), U1.31 (VSS), U1.47 (VSS), U1.63 (VSS), U1.7 (NRST), SW2.2, U119.2 (VO)
- net at U1.60 (BOOT0): now also R7.1
- net LEDDATA: now reaches U1.9 (PC1)
- net LEDDATA: now also U2.3 (DI)
- removed net +5V: R1.1, R1.2, SW1.1 (A)
- net I2C1_SCL: no longer names the net of U1.6 (PF1)
- net I2C1_SDA: no longer names the net of U1.5 (PF0)
- new net: U10.3 (DI), U2.1 (DO)
- new net: U10.1 (DO), U18.3 (DI)
- new net: U18.1 (DO), U26.3 (DI)
- new net: U26.1 (DO), U34.3 (DI)
- new net: U34.1 (DO), U42.3 (DI)
- new net: U42.1 (DO), U50.3 (DI)
- new net: U50.1 (DO), U58.3 (DI)
- new net: U58.1 (DO), U66.3 (DI)
- new net: U66.1 (DO), U74.3 (DI)
- new net: U74.1 (DO), U82.3 (DI)
- new net: U82.1 (DO), U90.3 (DI)
- new net: U90.1 (DO), U98.3 (DI)
- new net: U3.3 (DI), U98.1 (DO)
- new net: U11.3 (DI), U3.1 (DO)
- new net: U11.1 (DO), U19.3 (DI)
- new net: U19.1 (DO), U27.3 (DI)
- new net: U27.1 (DO), U35.3 (DI)
- new net: U35.1 (DO), U43.3 (DI)
- new net: U43.1 (DO), U51.3 (DI)
- new net: U51.1 (DO), U59.3 (DI)
- new net: U59.1 (DO), U67.3 (DI)
- new net: U67.1 (DO), U75.3 (DI)
- new net: U75.1 (DO), U83.3 (DI)
- new net: U83.1 (DO), U91.3 (DI)
- new net: U91.1 (DO), U99.3 (DI)
- new net: U4.3 (DI), U99.1 (DO)
- new net: U12.3 (DI), U4.1 (DO)
- new net: U12.1 (DO), U20.3 (DI)
- new net: U20.1 (DO), U28.3 (DI)
- new net: U28.1 (DO), U36.3 (DI)
- new net: U36.1 (DO), U44.3 (DI)
- new net: U44.1 (DO), U52.3 (DI)
- new net: U52.1 (DO), U60.3 (DI)
- new net: U60.1 (DO), U68.3 (DI)
- new net: U68.1 (DO), U76.3 (DI)
- new net: U76.1 (DO), U84.3 (DI)
- new net: U84.1 (DO), U92.3 (DI)
- new net: U100.3 (DI), U92.1 (DO)
- new net: U100.1 (DO), U5.3 (DI)
- new net: U13.3 (DI), U5.1 (DO)
- new net: U13.1 (DO), U21.3 (DI)
- new net: U21.1 (DO), U29.3 (DI)
- new net: U29.1 (DO), U37.3 (DI)
- new net: U37.1 (DO), U45.3 (DI)
- new net: U45.1 (DO), U53.3 (DI)
- new net: U53.1 (DO), U61.3 (DI)
- new net: U61.1 (DO), U69.3 (DI)
- new net: U69.1 (DO), U77.3 (DI)
- new net: U77.1 (DO), U85.3 (DI)
- new net: U85.1 (DO), U93.3 (DI)
- new net: U101.3 (DI), U93.1 (DO)
- new net: U101.1 (DO), U6.3 (DI)
- new net: U14.3 (DI), U6.1 (DO)
- new net: U14.1 (DO), U22.3 (DI)
- new net: U22.1 (DO), U30.3 (DI)
- new net: U30.1 (DO), U38.3 (DI)
- new net: U38.1 (DO), U46.3 (DI)
- new net: U46.1 (DO), U54.3 (DI)
- new net: U54.1 (DO), U62.3 (DI)
- new net: U62.1 (DO), U70.3 (DI)
- new net: U70.1 (DO), U78.3 (DI)
- new net: U78.1 (DO), U86.3 (DI)
- new net: U86.1 (DO), U94.3 (DI)
- new net: U102.3 (DI), U94.1 (DO)
- new net: U102.1 (DO), U7.3 (DI)
- new net: U15.3 (DI), U7.1 (DO)
- new net: U15.1 (DO), U23.3 (DI)
- new net: U23.1 (DO), U31.3 (DI)
- new net: U31.1 (DO), U39.3 (DI)
- new net: U39.1 (DO), U47.3 (DI)
- new net: U47.1 (DO), U55.3 (DI)
- new net: U55.1 (DO), U63.3 (DI)
- new net: U63.1 (DO), U71.3 (DI)
- new net: U71.1 (DO), U79.3 (DI)
- new net: U79.1 (DO), U87.3 (DI)
- new net: U87.1 (DO), U95.3 (DI)
- new net: U103.3 (DI), U95.1 (DO)
- new net: U103.1 (DO), U8.3 (DI)
- new net: U16.3 (DI), U8.1 (DO)
- new net: U104.4 (VDD), U105.4 (VDD), U106.4 (VDD), U107.4 (VDD), U108.4 (VDD), U109.4 (VDD), U110.4 (VDD), U111.4 (VDD), U112.4 (VDD), U113.4 (VDD), U114.4 (VDD), U115.4 (VDD), U116.4 (VDD), U117.4 (VDD), U118.4 (VDD), U16.4 (VDD), U17.4 (VDD), U24.4 (VDD), U25.4 (VDD), U32.4 (VDD), U33.4 (VDD), U40.4 (VDD), U41.4 (VDD), U48.4 (VDD), U49.4 (VDD), U56.4 (VDD), U57.4 (VDD), U64.4 (VDD), U65.4 (VDD), U72.4 (VDD), U73.4 (VDD), U8.4 (VDD), U80.4 (VDD), U81.4 (VDD), U88.4 (VDD), U89.4 (VDD), U9.4 (VDD), U96.4 (VDD), U97.4 (VDD)
- new net: U16.1 (DO), U24.3 (DI)
- new net: U24.1 (DO), U32.3 (DI)
- new net: U32.1 (DO), U40.3 (DI)
- new net: U40.1 (DO), U48.3 (DI)
- new net: U48.1 (DO), U56.3 (DI)
- new net: U56.1 (DO), U64.3 (DI)
- new net: U64.1 (DO), U72.3 (DI)
- new net: U72.1 (DO), U80.3 (DI)
- new net: U80.1 (DO), U88.3 (DI)
- new net: U88.1 (DO), U96.3 (DI)
- new net: U104.3 (DI), U96.1 (DO)
- new net: U104.1 (DO), U9.3 (DI)
- new net: U17.3 (DI), U9.1 (DO)
- new net: U17.1 (DO), U25.3 (DI)
- new net: U25.1 (DO), U33.3 (DI)
- new net: U33.1 (DO), U41.3 (DI)
- new net: U41.1 (DO), U49.3 (DI)
- new net: U49.1 (DO), U57.3 (DI)
- new net: U57.1 (DO), U65.3 (DI)
- new net: U65.1 (DO), U73.3 (DI)
- new net: U73.1 (DO), U81.3 (DI)
- new net: U81.1 (DO), U89.3 (DI)
- new net: U89.1 (DO), U97.3 (DI)
- new net: U105.3 (DI), U97.1 (DO)
- new net: U105.1 (DO), U106.3 (DI)
- new net: R6.1, SW2.1
- new net: U106.1 (DO), U107.3 (DI)
- new net: U107.1 (DO), U108.3 (DI)
- new net: U108.1 (DO), U109.3 (DI)
- new net: U109.1 (DO), U110.3 (DI)
- new net: U110.1 (DO), U111.3 (DI)
- new net: U111.1 (DO), U112.3 (DI)
- new net: U112.1 (DO), U113.3 (DI)
- new net: U113.1 (DO), U114.3 (DI)
- new net: U114.1 (DO), U115.3 (DI)
- new net: U115.1 (DO), U116.3 (DI)
- new net: U116.1 (DO), U117.3 (DI)
- new net: U117.1 (DO), U118.3 (DI)
- no-connect marks 0 -> 27
Other:
- note removed: "23 pins free for matrix input - 132 keys MAX"

Commit message: routed with all leds + gerbers
Changed lines of the file:
@@
-	1    0    0    -1
-$EndComp
-$Comp
-L power:PWR_FLAG #FLG0102
-U 1 1 5F0473D4
-P 2450 4250
-F 0 "#FLG0102" H 2450 4325 50  0001 C CNN
-F 1 "PWR_FLAG" H 2450 4423 50  0000 C CNN
-F 2 "" H 2450 4250 50  0001 C CNN
-F 3 "~" H 2450 4250 50  0001 C CNN
-	1    2450 4250
 	1    0    0    -1
 $EndComp
@@
 	0    -1   -1   0
 $EndComp
-Connection ~ 2450 4250
 $Comp
 L MCU_ST_STM32F0:STM32F070RBTx U1
